File: hardware/coupon/rev-a/rgb-badge-coupon.kicad_sch (KiCad schematic)
At the start: 0 parts

Commit message: Capture the 256-LED coupon matrix and verify pin-to-net assignments
Other:
- added sheet Rows 00-07, columns 00-07 (matrix-r00-c00.kicad_sch)
- added sheet Rows 00-07, columns 08-15 (matrix-r00-c08.kicad_sch)
- added sheet Rows 08-15, columns 00-07 (matrix-r08-c00.kicad_sch)
- added sheet Rows 08-15, columns 08-15 (matrix-r08-c08.kicad_sch)
- note added: "16 x 16 RGB matrix - initial circuit capture"
- note added: "EAST10105RGBA0 - 64 LEDs"
- note added: "Four sheets use global nets: ROW_00_A..ROW_15_A and COL_00_R/G/B..COL_15_R/G/B."
- note added: "No PCB placement exists. QBLP1515 rotation belongs to the later PCB, per ADR 0008."
- note added: "QBLP1515A-RGB2A - 64 LEDs"
- note added: "TLC59581, row stages, controller, USB and power circuits are not captured yet."
- note added: "These are 16 switched anodes and 48 cathode sinks. They are not logic control signals."
- title: (none) -> Coupon Rev A - matrix capture
Changed lines of the file:
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@@
 (kicad_sch
-	(version 20260306)
-	(generator "eeschema")
-	(generator_version "10.0")
-	(paper "A4")
-	(sheet_instances
-		(path "/"
-			(page "1")
-		)
-	)
-	(embedded_fonts no)
+(version 20260306)
+(generator "rgb_badge_matrix")
+(generator_version "1.0")
+(paper "A4")
+(title_block (title "Coupon Rev A - matrix capture") (rev "A - matrix draft") (comment 1 "SPDX-License-Identifier: CERN-OHL-S-2.0") (comment 2 "Matrix only: driver, row stages and power circuits pending"))
+(text "16 x 16 RGB matrix - initial circuit capture" (at 20.32 20.32 0) (effects (font (size 2.0 2.0)) (justify left)))
+(text "Four sheets use global nets: ROW_00_A..ROW_15_A and COL_00_R/G/B..COL_15_R/G/B." (at 20.32 30.48 0) (effects (font (size 1.27 1.27)) (justify left)))
+(text "These are 16 switched anodes and 48 cathode sinks. They are not logic control signals." (at 20.32 38.10 0) (effects (font (size 1.27 1.27)) (justify left)))
+(text "TLC59581, row stages, controller, USB and power circuits are not captured yet." (at 20.32 45.72 0) (effects (font (size 1.27 1.27)) (justify left)))
+(text "No PCB placement exists. QBLP1515 rotation belongs to the later PCB, per ADR 0008." (at 20.32 157.48 0) (effects (font (size 1.27 1.27)) (justify left)))
+(sheet (at 20.32 63.50) (size 116.84 27.94)
+(exclude_from_sim no) (in_bom yes) (on_board yes) (dnp no)
+(stroke (width 0.1524) (type solid)) (fill (color 0 0 0 0))
+(property "Sheetname" "Rows 00-07, columns 00-07" (at 20.32 62.23 0) (effects (font (size 1.27 1.27)) (justify left bottom)))
+(property "Sheetfile" "matrix-r00-c00.kicad_sch" (at 20.32 92.71 0) (effects (font (size 1.27 1.27)) (justify left top)))
+(instances (project "rgb-badge-coupon" (path "/207fb68e-2ddb-46bb-8712-eba2f8c5eef6" (page "2")))))
+(text "EAST10105RGBA0 - 64 LEDs" (at 25.40 76.20 0) (effects (font (size 1.27 1.27)) (justify left)))
+(sheet (at 152.40 63.50) (size 116.84 27.94)
+(exclude_from_sim no) (in_bom yes) (on_board yes) (dnp no)
+(stroke (width 0.1524) (type solid)) (fill (color 0 0 0 0))
+(property "Sheetname" "Rows 00-07, columns 08-15" (at 152.40 62.23 0) (effects (font (size 1.27 1.27)) (justify left bottom)))
+(property "Sheetfile" "matrix-r00-c08.kicad_sch" (at 152.40 92.71 0) (effects (font (size 1.27 1.27)) (justify left top)))
+(instances (project "rgb-badge-coupon" (path "/207fb68e-2ddb-46bb-8712-eba2f8c5eef6" (page "3")))))
+(text "QBLP1515A-RGB2A - 64 LEDs" (at 157.48 76.20 0) (effects (font (size 1.27 1.27)) (justify left)))
+(sheet (at 20.32 109.22) (size 116.84 27.94)
+(exclude_from_sim no) (in_bom yes) (on_board yes) (dnp no)
+(stroke (width 0.1524) (type solid)) (fill (color 0 0 0 0))
+(property "Sheetname" "Rows 08-15, columns 00-07" (at 20.32 107.95 0) (effects (font (size 1.27 1.27)) (justify left bottom)))
+(property "Sheetfile" "matrix-r08-c00.kicad_sch" (at 20.32 138.43 0) (effects (font (size 1.27 1.27)) (justify left top)))
+(instances (project "rgb-badge-coupon" (path "/207fb68e-2ddb-46bb-8712-eba2f8c5eef6" (page "4")))))
+(text "EAST10105RGBA0 - 64 LEDs" (at 25.40 121.92 0) (effects (font (size 1.27 1.27)) (justify left)))
+(sheet (at 152.40 109.22) (size 116.84 27.94)
+(exclude_from_sim no) (in_bom yes) (on_board yes) (dnp no)
+(stroke (width 0.1524) (type solid)) (fill (color 0 0 0 0))
+(property "Sheetname" "Rows 08-15, columns 08-15" (at 152.40 107.95 0) (effects (font (size 1.27 1.27)) (justify left bottom)))
+(property "Sheetfile" "matrix-r08-c08.kicad_sch" (at 152.40 138.43 0) (effects (font (size 1.27 1.27)) (justify left top)))
+(instances (project "rgb-badge-coupon" (path "/207fb68e-2ddb-46bb-8712-eba2f8c5eef6" (page "5")))))
+(text "QBLP1515A-RGB2A - 64 LEDs" (at 157.48 121.92 0) (effects (font (size 1.27 1.27)) (justify left)))
+(sheet_instances (path "/" (page "1")))
+(embedded_fonts no)
 )
