File: hardware/coupon/rev-a/rgb-badge-coupon.kicad_sch (KiCad schematic)
At the start: 0 parts

Commit message: Link dark VLED converter stage into coupon schematic
Other:
- added sheet Provisional dark VLED converter (vled-converter.kicad_sch)
- note added: "E0/E1/BQ, application 3V3 and dark VLED stage captured; pack and VLED interlock pending."
- note removed: "USB logic, provisional E0/E1/BQ, and application 3V3 staged; pack and VLED pending."
Changed lines of the file:
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@@
 (generator_version "1.0")
 (paper "A2")
-(title_block (title "Coupon Rev A - display, USB and provisional power") (rev "A-draft") (comment 1 "SPDX-License-Identifier: CERN-OHL-S-2.0") (comment 2 "Pack, gauge switch and VLED pending; E0/E1 unqualified"))
+(title_block (title "Coupon Rev A - display, USB and provisional power") (rev "A-draft") (comment 1 "SPDX-License-Identifier: CERN-OHL-S-2.0") (comment 2 "Pack, gauge switch and VLED interlock pending; E0/E1 unqualified"))
 (text "16 x 16 RGB matrix, TLC59581 driver, row selectors and ESP32-S3 controller" (at 20.32 20.32 0) (effects (font (size 2.0 2.0)) (justify left)))
 (text "Four sheets use global nets: ROW_00_A..ROW_15_A and COL_00_R/G/B..COL_15_R/G/B." (at 20.32 30.48 0) (effects (font (size 1.27 1.27)) (justify left)))
 (text "These are 16 switched anodes and 48 cathode sinks. They are not logic control signals." (at 20.32 38.10 0) (effects (font (size 1.27 1.27)) (justify left)))
-(text "USB logic, provisional E0/E1/BQ, and application 3V3 staged; pack and VLED pending." (at 20.32 45.72 0) (effects (font (size 1.27 1.27)) (justify left)))
+(text "E0/E1/BQ, application 3V3 and dark VLED stage captured; pack and VLED interlock pending." (at 20.32 45.72 0) (effects (font (size 1.27 1.27)) (justify left)))
 (text "No PCB yet. QBLP1515 rotation: ADR 0008. Never fabricate before Gate A." (at 20.32 273.05 0) (effects (font (size 1.27 1.27)) (justify left)))
 (sheet (at 20.32 63.50) (size 116.84 27.94)
@@
 (property "Sheetfile" "usb-protection.kicad_sch" (at 152.40 321.31 0) (effects (font (size 1.27 1.27)) (justify left top)))
 (instances (project "rgb-badge-coupon" (path "/207fb68e-2ddb-46bb-8712-eba2f8c5eef6" (page "18")))))
+(sheet (at 284.48 297.18) (size 116.84 22.86)
+(exclude_from_sim no) (in_bom yes) (on_board yes) (dnp no)
+(stroke (width 0.1524) (type solid)) (fill (color 0 0 0 0))
+(property "Sheetname" "Provisional dark VLED converter" (at 284.48 295.91 0) (effects (font (size 1.27 1.27)) (justify left bottom)))
+(property "Sheetfile" "vled-converter.kicad_sch" (at 284.48 321.31 0) (effects (font (size 1.27 1.27)) (justify left top)))
+(instances (project "rgb-badge-coupon" (path "/207fb68e-2ddb-46bb-8712-eba2f8c5eef6" (page "19")))))
 (sheet_instances (path "/" (page "1")))
 (embedded_fonts no)

Commit message: Capture output-isolated display interlock and screen complete fit
Other:
- added sheet Display interlock (output-isolated trial) (display-interlock.kicad_sch)
- note added: "E0/E1/BQ, app 3V3, dark VLED and output-isolated interlock captured; fault qualification pending."
- note removed: "E0/E1/BQ, application 3V3 and dark VLED stage captured; pack and VLED interlock pending."
Changed lines of the file:
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@@
 (generator_version "1.0")
 (paper "A2")
-(title_block (title "Coupon Rev A - display, USB and provisional power") (rev "A-draft") (comment 1 "SPDX-License-Identifier: CERN-OHL-S-2.0") (comment 2 "Pack, gauge switch and VLED interlock pending; E0/E1 unqualified"))
+(title_block (title "Coupon Rev A - display, USB and provisional power") (rev "A-draft") (comment 1 "SPDX-License-Identifier: CERN-OHL-S-2.0") (comment 2 "Interlock outputs isolated; E0/E1 and board unqualified"))
 (text "16 x 16 RGB matrix, TLC59581 driver, row selectors and ESP32-S3 controller" (at 20.32 20.32 0) (effects (font (size 2.0 2.0)) (justify left)))
 (text "Four sheets use global nets: ROW_00_A..ROW_15_A and COL_00_R/G/B..COL_15_R/G/B." (at 20.32 30.48 0) (effects (font (size 1.27 1.27)) (justify left)))
 (text "These are 16 switched anodes and 48 cathode sinks. They are not logic control signals." (at 20.32 38.10 0) (effects (font (size 1.27 1.27)) (justify left)))
-(text "E0/E1/BQ, application 3V3 and dark VLED stage captured; pack and VLED interlock pending." (at 20.32 45.72 0) (effects (font (size 1.27 1.27)) (justify left)))
+(text "E0/E1/BQ, app 3V3, dark VLED and output-isolated interlock captured; fault qualification pending." (at 20.32 45.72 0) (effects (font (size 1.27 1.27)) (justify left)))
 (text "No PCB yet. QBLP1515 rotation: ADR 0008. Never fabricate before Gate A." (at 20.32 273.05 0) (effects (font (size 1.27 1.27)) (justify left)))
 (sheet (at 20.32 63.50) (size 116.84 27.94)
@@
 (property "Sheetfile" "vled-converter.kicad_sch" (at 284.48 321.31 0) (effects (font (size 1.27 1.27)) (justify left top)))
 (instances (project "rgb-badge-coupon" (path "/207fb68e-2ddb-46bb-8712-eba2f8c5eef6" (page "19")))))
+(sheet (at 416.56 63.50) (size 116.84 22.86)
+(exclude_from_sim no) (in_bom yes) (on_board yes) (dnp no)
+(stroke (width 0.1524) (type solid)) (fill (color 0 0 0 0))
+(property "Sheetname" "Display interlock (output-isolated trial)" (at 416.56 62.23 0) (effects (font (size 1.27 1.27)) (justify left bottom)))
+(property "Sheetfile" "display-interlock.kicad_sch" (at 416.56 87.63 0) (effects (font (size 1.27 1.27)) (justify left top)))
+(instances (project "rgb-badge-coupon" (path "/207fb68e-2ddb-46bb-8712-eba2f8c5eef6" (page "20")))))
 (sheet_instances (path "/" (page "1")))
 (embedded_fonts no)
