File: hardware/coupon/rev-a/charger-gate.kicad_sch (KiCad schematic)
At the start: 11 parts, among them U42 SN74AUP1G125DBVR, U43 SN74AUP1G125DBVR, U44 TPS259474ARPWR

Commit message: Capture provisional E0 protected USB source bridge
Connections:
- net USB_PROTECTED_DRAFT renamed +5V_USB
Other:
- note added: "E1 IN joins E0 protected +5V_USB; E1 OUT joins BQ IN and EN2 clamp."
- note removed: "E1 IN is a draft protected-USB boundary. E1 OUT joins BQ IN and EN2 clamp."
Changed lines of the file:
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@@
 (generator_version "1.0")
 (paper "A3")
-(title_block (title "Coupon Rev A - provisional E1 charger gate") (rev "A-draft") (comment 1 "SPDX-License-Identifier: CERN-OHL-S-2.0") (comment 2 "E0 upstream source still absent; gate operating behavior unqualified"))
-(text "E1 IN is a draft protected-USB boundary. E1 OUT joins BQ IN and EN2 clamp." (at 20.320 20.320 0) (effects (font (size 1.27 1.27)) (justify left)))
+(title_block (title "Coupon Rev A - provisional E1 charger gate") (rev "A-draft") (comment 1 "SPDX-License-Identifier: CERN-OHL-S-2.0") (comment 2 "E0 source captured; gate operating behavior unqualified"))
+(text "E1 IN joins E0 protected +5V_USB; E1 OUT joins BQ IN and EN2 clamp." (at 20.320 20.320 0) (effects (font (size 1.27 1.27)) (justify left)))
 (text "Three AUP sinks: source request, supervisor RESET, and temperature on the other sheet." (at 20.320 27.940 0) (effects (font (size 1.27 1.27)) (justify left)))
 (text "Static divider screen assumes 1.6uA leakage; no startup, inrush or E0 fault qualification." (at 20.320 35.560 0) (effects (font (size 1.27 1.27)) (justify left)))
@@
 (instances (project "rgb-badge-coupon" (path "/207fb68e-2ddb-46bb-8712-eba2f8c5eef6/d8d1f8f8-44be-5ad4-a193-9dc90529f25a" (reference "C59") (unit 1)))))
 (wire (pts (xy 154.940 96.520) (xy 124.460 96.520)) (stroke (width 0) (type default)))
-(global_label "USB_PROTECTED_DRAFT" (shape passive) (at 124.460 96.520 180) (effects (font (size 1.27 1.27)) (justify right)) (property "Intersheetrefs" "${INTERSHEET_REFS}" (at 124.460 96.520 0) (effects (font (size 1.27 1.27)) (hide yes))))
+(global_label "+5V_USB" (shape passive) (at 124.460 96.520 180) (effects (font (size 1.27 1.27)) (justify right)) (property "Intersheetrefs" "${INTERSHEET_REFS}" (at 124.460 96.520 0) (effects (font (size 1.27 1.27)) (hide yes))))
 (wire (pts (xy 154.940 101.600) (xy 124.460 101.600)) (stroke (width 0) (type default)))
 (global_label "CHARGER_GATE_EN" (shape passive) (at 124.460 101.600 180) (effects (font (size 1.27 1.27)) (justify right)) (property "Intersheetrefs" "${INTERSHEET_REFS}" (at 124.460 101.600 0) (effects (font (size 1.27 1.27)) (hide yes))))
@@
 (global_label "GND" (shape passive) (at 279.400 132.080 0) (effects (font (size 1.27 1.27)) (justify left)) (property "Intersheetrefs" "${INTERSHEET_REFS}" (at 279.400 132.080 0) (effects (font (size 1.27 1.27)) (hide yes))))
 (wire (pts (xy 71.120 111.760) (xy 50.800 111.760)) (stroke (width 0) (type default)))
-(global_label "USB_PROTECTED_DRAFT" (shape passive) (at 50.800 111.760 180) (effects (font (size 1.27 1.27)) (justify right)) (property "Intersheetrefs" "${INTERSHEET_REFS}" (at 50.800 111.760 0) (effects (font (size 1.27 1.27)) (hide yes))))
+(global_label "+5V_USB" (shape passive) (at 50.800 111.760 180) (effects (font (size 1.27 1.27)) (justify right)) (property "Intersheetrefs" "${INTERSHEET_REFS}" (at 50.800 111.760 0) (effects (font (size 1.27 1.27)) (hide yes))))
 (wire (pts (xy 81.280 111.760) (xy 101.600 111.760)) (stroke (width 0) (type default)))
 (global_label "GND" (shape passive) (at 101.600 111.760 0) (effects (font (size 1.27 1.27)) (justify left)) (property "Intersheetrefs" "${INTERSHEET_REFS}" (at 101.600 111.760 0) (effects (font (size 1.27 1.27)) (hide yes))))
@@
 (wire (pts (xy 259.080 223.520) (xy 279.400 223.520)) (stroke (width 0) (type default)))
 (global_label "GND" (shape passive) (at 279.400 223.520 0) (effects (font (size 1.27 1.27)) (justify left)) (property "Intersheetrefs" "${INTERSHEET_REFS}" (at 279.400 223.520 0) (effects (font (size 1.27 1.27)) (hide yes))))
-(symbol (lib_id "rgb-badge-coupon:PWR_FLAG") (at 76.200 157.480 0) (unit 1)
-(exclude_from_sim no) (in_bom no) (on_board no) (dnp no)
-(property "Reference" "#FLG08" (at 76.200 152.400 0) (effects (font (size 1.27 1.27))))
-(property "Value" "PWR_FLAG" (at 76.200 154.940 0) (effects (font (size 1.27 1.27))))
-(property "Footprint" "" (at 76.200 157.480 0) (effects (font (size 1.27 1.27)) (hide yes)))
-(property "Datasheet" "" (at 76.200 157.480 0) (effects (font (size 1.27 1.27)) (hide yes)))
-(property "Manufacturer" "" (at 76.200 157.480 0) (effects (font (size 1.27 1.27)) (hide yes)))
-(property "MPN" "" (at 76.200 157.480 0) (effects (font (size 1.27 1.27)) (hide yes)))
-(pin "1")
-(instances (project "rgb-badge-coupon" (path "/207fb68e-2ddb-46bb-8712-eba2f8c5eef6/d8d1f8f8-44be-5ad4-a193-9dc90529f25a" (reference "#FLG08") (unit 1)))))
-(wire (pts (xy 76.200 157.480) (xy 96.520 157.480)) (stroke (width 0) (type default)))
-(global_label "USB_PROTECTED_DRAFT" (shape passive) (at 96.520 157.480 0) (effects (font (size 1.27 1.27)) (justify left)) (property "Intersheetrefs" "${INTERSHEET_REFS}" (at 96.520 157.480 0) (effects (font (size 1.27 1.27)) (hide yes))))
 (embedded_fonts no)
 )
