File: hardware/coupon/rev-a/gauge.kicad_sch (KiCad schematic)
At the start: 4 parts, among them U35 MAX17048G+T10

Commit message: Normalize Panasonic ERJ order codes across coupon
Parts:
- R79, R80: symbol rgb-badge-coupon:ERJ-2RKF2201X -> rgb-badge-coupon:ERJ2RKF2201X; MPN ERJ-2RKF2201X -> ERJ2RKF2201X
Changed lines of the file:
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@@
 (global_label "SYS_I2C_SCL" (shape passive) (at 134.620 83.820 0) (effects (font (size 1.27 1.27)) (justify left)) (property "Intersheetrefs" "${INTERSHEET_REFS}" (at 134.620 83.820 0) (effects (font (size 1.27 1.27)) (hide yes))))
 (no_connect (at 111.760 76.200))
-(symbol (lib_id "rgb-badge-coupon:ERJ-2RKF2201X") (at 198.120 71.120 0) (unit 1)
+(symbol (lib_id "rgb-badge-coupon:ERJ2RKF2201X") (at 198.120 71.120 0) (unit 1)
 (exclude_from_sim no) (in_bom yes) (on_board yes) (dnp no)
 (property "Reference" "R79" (at 198.120 66.040 0) (effects (font (size 1.27 1.27))))
@@
 (property "Datasheet" "https://industrial.panasonic.com/cdbs/www-data/pdf/RDA0000/AOA0000C304.pdf" (at 198.120 71.120 0) (effects (font (size 1.27 1.27)) (hide yes)))
 (property "Manufacturer" "Panasonic" (at 198.120 71.120 0) (effects (font (size 1.27 1.27)) (hide yes)))
-(property "MPN" "ERJ-2RKF2201X" (at 198.120 71.120 0) (effects (font (size 1.27 1.27)) (hide yes)))
+(property "MPN" "ERJ2RKF2201X" (at 198.120 71.120 0) (effects (font (size 1.27 1.27)) (hide yes)))
 (pin "1")
 (pin "2")
@@
 (wire (pts (xy 203.200 71.120) (xy 218.440 71.120)) (stroke (width 0) (type default)))
 (global_label "SYS_I2C_SDA" (shape passive) (at 218.440 71.120 0) (effects (font (size 1.27 1.27)) (justify left)) (property "Intersheetrefs" "${INTERSHEET_REFS}" (at 218.440 71.120 0) (effects (font (size 1.27 1.27)) (hide yes))))
-(symbol (lib_id "rgb-badge-coupon:ERJ-2RKF2201X") (at 198.120 91.440 0) (unit 1)
+(symbol (lib_id "rgb-badge-coupon:ERJ2RKF2201X") (at 198.120 91.440 0) (unit 1)
 (exclude_from_sim no) (in_bom yes) (on_board yes) (dnp no)
 (property "Reference" "R80" (at 198.120 86.360 0) (effects (font (size 1.27 1.27))))
@@
 (property "Datasheet" "https://industrial.panasonic.com/cdbs/www-data/pdf/RDA0000/AOA0000C304.pdf" (at 198.120 91.440 0) (effects (font (size 1.27 1.27)) (hide yes)))
 (property "Manufacturer" "Panasonic" (at 198.120 91.440 0) (effects (font (size 1.27 1.27)) (hide yes)))
-(property "MPN" "ERJ-2RKF2201X" (at 198.120 91.440 0) (effects (font (size 1.27 1.27)) (hide yes)))
+(property "MPN" "ERJ2RKF2201X" (at 198.120 91.440 0) (effects (font (size 1.27 1.27)) (hide yes)))
 (pin "1")
 (pin "2")

Commit message: Connect switched gauge through isolated I2C buffer
Parts:
- added C64, C65: 100n 16V X7R, rgb-badge-coupon:C_Murata_GRM15_0402, symbol rgb-badge-coupon:GRM155R71C104KA88D
- added R101, R102: 2.2k 1%, rgb-badge-coupon:R_Panasonic_ERJ2_0402, symbol rgb-badge-coupon:ERJ2RKF2201X
- added U46: TCA9517ADGKR, rgb-badge-coupon:VSSOP_TI_DGK0008A, symbol rgb-badge-coupon:TCA9517ADGKR
Connections:
- net +3V3_APP: now also C65.1, U46.5 (EN), U46.8 (VCCB)
- net +BAT_GAUGE_SW: now also C64.1, R101.1, R102.1, U46.1 (VCCA)
- net GND: now also C64.2, C65.2, U46.4 (GND)
- net SYS_I2C_SCL: now also U46.7 (SCLB); no longer U35.7 (SCL)
- net SYS_I2C_SDA: now also U46.6 (SDAB); no longer U35.8 (SDA)
- new net GAUGE_I2C_SCL: R102.2, U35.7 (SCL), U46.2 (SCLA)
- new net GAUGE_I2C_SDA: R101.2, U35.8 (SDA), U46.3 (SDAA)
Other:
- note added: "MAX17048 and TCA9517A port A share switched BAT. Port B joins 3V3 application I2C."
- note added: "PWR_FLAG marks switched BAT through SW2 for ERC. Contact bounce and rail decay remain unqualified."
- note removed: "MAX17048: switched gauge domain; no charger, pack, or mechanical switch here"
- note removed: "PWR_FLAG is a temporary switched-BAT source assumption, NOT a physical connection."
- title: Coupon Rev A - staged switched fuel gauge -> Coupon Rev A - switched fuel gauge and I2C buffer
