File: hardware/coupon/rev-a/charger-core.kicad_sch (KiCad schematic)
At the start: 9 parts, among them J2 S2B-PH-SM4-TB, U38 2.5V shunt, U41 BQ24074RGTR

Commit message: Correct all six exact Murata capacitor lands and preserve 59-edge routing
Parts:
- C53, C54: footprint rgb-badge-coupon:C_Murata_GRM18_0603 -> rgb-badge-coupon:C_Murata_GRM188R60J106ME47_0603
Changed lines of the file:
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@@
 (property "Reference" "C53" (at 254.000 69.850 0) (effects (font (size 1.27 1.27))))
 (property "Value" "10u 6.3V X5R" (at 254.000 72.390 0) (effects (font (size 1.27 1.27))))
-(property "Footprint" "rgb-badge-coupon:C_Murata_GRM18_0603" (at 254.000 76.200 0) (effects (font (size 1.27 1.27)) (hide yes)))
+(property "Footprint" "rgb-badge-coupon:C_Murata_GRM188R60J106ME47_0603" (at 254.000 76.200 0) (effects (font (size 1.27 1.27)) (hide yes)))
 (property "Datasheet" "https://pim.murata.com/en-global/pim/details/?partNum=GRM188R60J106ME47D" (at 254.000 76.200 0) (effects (font (size 1.27 1.27)) (hide yes)))
 (property "Manufacturer" "Murata" (at 254.000 76.200 0) (effects (font (size 1.27 1.27)) (hide yes)))
@@
 (property "Reference" "C54" (at 254.000 90.170 0) (effects (font (size 1.27 1.27))))
 (property "Value" "10u 6.3V X5R" (at 254.000 92.710 0) (effects (font (size 1.27 1.27))))
-(property "Footprint" "rgb-badge-coupon:C_Murata_GRM18_0603" (at 254.000 96.520 0) (effects (font (size 1.27 1.27)) (hide yes)))
+(property "Footprint" "rgb-badge-coupon:C_Murata_GRM188R60J106ME47_0603" (at 254.000 96.520 0) (effects (font (size 1.27 1.27)) (hide yes)))
 (property "Datasheet" "https://pim.murata.com/en-global/pim/details/?partNum=GRM188R60J106ME47D" (at 254.000 96.520 0) (effects (font (size 1.27 1.27)) (hide yes)))
 (property "Manufacturer" "Murata" (at 254.000 96.520 0) (effects (font (size 1.27 1.27)) (hide yes)))
