File: hardware/coupon/rev-a/staging/vled-routing-trial.kicad_pcb (KiCad board)
At the start: 2 copper layers, 15 x 10.5 mm, 13 parts, among them U37 TPS63020DSJT

Commit message: Reorder VLED feedback divider in fit and KiCad trials
Parts:
- moved R84 4.30 mm to (98.5, 23.3), turned to 180 degrees
- moved R86 4.30 mm to (94.2, 23.3), turned to 180 degrees
- turned R85 to 180 degrees
Changed lines of the file:
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@@
 	(footprint "rgb-badge-coupon:R_Panasonic_ERJ2_0402"
 		(layer "F.Cu")
-		(at 94.25 23.3)
+		(at 98.55 23.3 180)
 		(descr "Manufacturer range-based reflow land pattern; SPDX-License-Identifier: CERN-OHL-S-2.0")
 		(property "Reference" "R84"
-			(at 0 -1 0)
+			(at 0 -1 180)
 			(layer "F.SilkS")
 			(hide yes)
@@
 		)
 		(property "Value" "620k 1%"
-			(at 0 1 0)
+			(at 0 1 180)
 			(layer "F.Fab")
 			(hide yes)
@@
 		)
 		(property "Datasheet" ""
-			(at 0 0 0)
+			(at 0 0 180)
 			(layer "F.Fab")
 			(hide yes)
@@
 		)
 		(property "Description" ""
-			(at 0 0 0)
+			(at 0 0 180)
 			(layer "F.Fab")
 			(hide yes)
@@
 		)
 		(pad "1" smd rect
-			(at -0.5 0)
+			(at -0.5 0 180)
 			(size 0.5 0.5)
 			(layers "F.Cu" "F.Mask" "F.Paste")
@@
 		)
 		(pad "2" smd rect
-			(at 0.5 0)
+			(at 0.5 0 180)
 			(size 0.5 0.5)
 			(layers "F.Cu" "F.Mask" "F.Paste")
@@
 	(footprint "rgb-badge-coupon:R_Panasonic_ERJ2_0402"
 		(layer "F.Cu")
-		(at 96.4 23.3)
+		(at 96.4 23.3 180)
 		(descr "Manufacturer range-based reflow land pattern; SPDX-License-Identifier: CERN-OHL-S-2.0")
 		(property "Reference" "R85"
-			(at 0 -1 0)
+			(at 0 -1 180)
 			(layer "F.SilkS")
 			(hide yes)
@@
 		)
 		(property "Value" "620k 1%"
-			(at 0 1 0)
+			(at 0 1 180)
 			(layer "F.Fab")
 			(hide yes)
@@
 		)
 		(property "Datasheet" ""
-			(at 0 0 0)
+			(at 0 0 180)
 			(layer "F.Fab")
 			(hide yes)
@@
 		)
 		(property "Description" ""
-			(at 0 0 0)
+			(at 0 0 180)
 			(layer "F.Fab")
 			(hide yes)
@@
 		)
 		(pad "1" smd rect
-			(at -0.5 0)
+			(at -0.5 0 180)
 			(size 0.5 0.5)
 			(layers "F.Cu" "F.Mask" "F.Paste")
@@
 		)
 		(pad "2" smd rect
-			(at 0.5 0)
+			(at 0.5 0 180)
 			(size 0.5 0.5)
 			(layers "F.Cu" "F.Mask" "F.Paste")
@@
 	(footprint "rgb-badge-coupon:R_Panasonic_ERJ2_0402"
 		(layer "F.Cu")
-		(at 98.55 23.3)
+		(at 94.25 23.3 180)
 		(descr "Manufacturer range-based reflow land pattern; SPDX-License-Identifier: CERN-OHL-S-2.0")
 		(property "Reference" "R86"
-			(at 0 -1 0)
+			(at 0 -1 180)
 			(layer "F.SilkS")
 			(hide yes)
@@
 		)
 		(property "Value" "180k 1%"
-			(at 0 1 0)
+			(at 0 1 180)
 			(layer "F.Fab")
 			(hide yes)
@@
 		)
 		(property "Datasheet" ""
-			(at 0 0 0)
+			(at 0 0 180)
 			(layer "F.Fab")
 			(hide yes)
@@
 		)
 		(property "Description" ""
-			(at 0 0 0)
+			(at 0 0 180)
 			(layer "F.Fab")
 			(hide yes)
@@
 		)
 		(pad "1" smd rect
-			(at -0.5 0)
+			(at -0.5 0 180)
 			(size 0.5 0.5)
 			(layers "F.Cu" "F.Mask" "F.Paste")
@@
 		)
 		(pad "2" smd rect
-			(at 0.5 0)
-			(size 0.5 0.5)
-			(layers "F.Cu" "F.Mask" "F.Paste")
+			(at 0.5 0 180)
+			(size 0.5 0.5)
+			(layers "F.Cu" "F.Mask" "F.Paste")
