File: hardware/coupon/rev-a/staging/full-coupon-placement-trial-120mm.kicad_pcb (KiCad board)
At the start: 6 copper layers, 120 x 32.5 mm, 497 parts, among them J1 USB4505-03-0-A, J2 S2B-PH-SM4-TB, Q1 DMP2066LSN-7, Q10 DMP2066LSN-7, Q11 DMP2066LSN-7, Q12 DMP2066LSN-7, Q13 DMP2066LSN-7, Q14 DMP2066LSN-7, Q15 DMP2066LSN-7, Q16 DMP2066LSN-7, Q17 2N7002K-7, Q18 2N7002K-7, Q19 2N7002K-7, Q2 DMP2066LSN-7, Q20 2N7002K-7, Q21 2N7002K-7, Q22 2N7002K-7, Q23 2N7002K-7, Q24 2N7002K-7, Q25 2N7002K-7, Q26 2N7002K-7, Q27 2N7002K-7, Q28 2N7002K-7, Q29 2N7002K-7, Q3 DMP2066LSN-7, Q30 2N7002K-7, Q31 2N7002K-7, Q32 2N7002K-7, Q4 DMP2066LSN-7, Q5 DMP2066LSN-7, Q6 DMP2066LSN-7, Q7 DMP2066LSN-7, Q8 DMP2066LSN-7, Q9 DMP2066LSN-7, SW1 EVQP7J01P, SW2 JS202011JCQN, U1 TLC59581RTQT, U11 SN74LVC1G04DBVR, U17 SN74LVC1G11DBVR, U2 74HC4514PW,118, U23 SN74LVC1G06DBVR, U24 SN74LVC2G17DBVR, U25 SN74LVC2G17DBVR, U29 TPS70933DBVR, U3 ESP32-S3-WROOM-1U-N16R8, U31 TUSB320LAIRWBR, U32 TS3USB31ERSER, U33 TPD4E05U06DQAR, U34 TPS3808G01DBVR, U35 MAX17048G+T10, U36 TPS631000DRLR, U37 TPS63020DSJT, U38 2.5V shunt, U39 TMP390A2DRLR, U40 SN74AUP1G125DBVR, U41 BQ24074RGTR, U42 SN74AUP1G125DBVR, U43 SN74AUP1G125DBVR, U44 TPS259474ARPWR, U45 TPS259474ARPWR, U46 TCA9517ADGKR, U47 TPS3823A-33DBVR, U48 SN74LVC1G04DSFR, U49 SN74LVC1G74RSER, U50 SN74LVC1G74RSER, U51 SN74LVC1G11DRYR, U52 SN74LVC1G08DSFR, U53 TLV6700DSER, U54 SN74LVC2G00DCUR, U55 SN74LVC2G08DCUR

Commit message: Connect eFuse output capacitor ground in placement study
Routing:
- net GND: track 35.2 -> 38.5 mm, vias 8 -> 9
Changed lines of the file:
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@@
+	)
+	(segment
+		(start 108.2 16)
+		(end 108.8 13.5)
+		(width 0.2)
+		(layer "In3.Cu")
+		(net "GND")
 	)
 	(segment
@@
 		(start 108.85 19)
 		(end 108.1 19)
+		(width 0.2)
+		(layer "B.Cu")
+		(net "GND")
+	)
+	(segment
+		(start 108.95 16)
+		(end 108.2 16)
 		(width 0.2)
 		(layer "B.Cu")
@@
 		(size 0.6)
 		(drill 0.3)
+		(layers "F.Cu" "B.Cu")
+		(net "GND")
+	)
+	(via
+		(at 108.2 16)
+		(size 0.6)
+		(drill 0.3)

Commit message: Connect USB eFuse timing capacitor grounds in staged board
Routing:
- net GND: track 38.5 -> 53.3 mm, vias 9 -> 11
Changed lines of the file:
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@@
+	)
+	(segment
+		(start 101.3 16)
+		(end 108.2 16)
+		(width 0.2)
+		(layer "In3.Cu")
+		(net "GND")
+	)
+	(segment
+		(start 101.3 19)
+		(end 108.1 19)
+		(width 0.2)
+		(layer "In3.Cu")
+		(net "GND")
+	)
+	(segment
+		(start 101.85 16)
+		(end 101.3 16)
+		(width 0.2)
+		(layer "B.Cu")
+		(net "GND")
+	)
+	(segment
+		(start 101.85 19)
+		(end 101.3 19)
+		(width 0.2)
+		(layer "B.Cu")
+		(net "GND")
 	)
 	(segment
@@
 	)
 	(via
+		(at 101.3 16)
+		(size 0.6)
+		(drill 0.3)
+		(layers "F.Cu" "B.Cu")
+		(net "GND")
+	)
+	(via
+		(at 101.3 19)
+		(size 0.6)
+		(drill 0.3)
+		(layers "F.Cu" "B.Cu")
+		(net "GND")
+	)
+	(via

Commit message: Join second USB ground and charger-gate ground pad
Routing:
- net GND: track 53.3 -> 60.6 mm, vias 11 -> 12
Changed lines of the file:
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@@
+	)
+	(segment
+		(start 106.65 18.775)
+		(end 107.2 18.775)
+		(width 0.2)
+		(layer "B.Cu")
+		(net "GND")
+	)
+	(segment
+		(start 107.2 18.775)
+		(end 108.1 19)
+		(width 0.2)
+		(layer "B.Cu")
+		(net "GND")
 	)
 	(segment
@@
 	)
 	(segment
+		(start 109 20)
+		(end 108.1 19)
+		(width 0.2)
+		(layer "In3.Cu")
+		(net "GND")
+	)
+	(segment
 		(start 109.5 12.5)
 		(end 110.2 13.2)
@@
 	)
 	(segment
+		(start 111.2 20)
+		(end 109 20)
+		(width 0.2)
+		(layer "In3.Cu")
+		(net "GND")
+	)
+	(segment
 		(start 112.2 15.2)
 		(end 110.2 13.2)
@@
 	)
 	(segment
+		(start 112.2 19.45)
+		(end 111.2 20)
+		(width 0.2)
+		(layer "F.Cu")
+		(net "GND")
+	)
+	(segment
 		(start 112.35 24.5)
 		(end 110.5 24.5)
@@
 		(layer "F.Cu")
 		(net "VBUS_CONNECTOR")
+	)
+	(segment
+		(start 113.25 19.45)
+		(end 112.2 19.45)
+		(width 0.2)
+		(layer "F.Cu")
+		(net "GND")
 	)
 	(segment
@@
 	)
 	(via
+		(at 111.2 20)
+		(size 0.6)
+		(drill 0.3)
+		(layers "F.Cu" "B.Cu")
+		(net "GND")
+	)
+	(via

Commit message: Connect both USB eFuse IC ground pins in staged board
Routing:
- net GND: track 60.6 -> 68.0 mm, vias 12 -> 14
- net E1_DVDT: track 2.53 -> 3.38 mm
Changed lines of the file:
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@@
+	)
+	(segment
+		(start 102 15.225)
+		(end 101.3 16)
+		(width 0.2)
+		(layer "In3.Cu")
+		(net "GND")
 	)
 	(segment
@@
 	(segment
 		(start 102.65 19)
-		(end 105.025 19.875)
+		(end 102.65 20)
+		(width 0.2)
+		(layer "B.Cu")
+		(net "E1_DVDT")
+	)
+	(segment
+		(start 102.65 20)
+		(end 104 20)
 		(width 0.2)
 		(layer "B.Cu")
@@
 	)
 	(segment
+		(start 103.4 19.3)
+		(end 101.3 19)
+		(width 0.2)
+		(layer "In3.Cu")
+		(net "GND")
+	)
+	(segment
 		(start 103.75 14)
 		(end 103.75 14.78)
@@
 		(layer "B.Cu")
 		(net "E1_ILM")
+	)
+	(segment
+		(start 104 20)
+		(end 105.025 19.875)
+		(width 0.2)
+		(layer "B.Cu")
+		(net "E1_DVDT")
+	)
+	(segment
+		(start 104.85 15.225)
+		(end 102 15.225)
+		(width 0.2)
+		(layer "B.Cu")
+		(net "GND")
+	)
+	(segment
+		(start 104.85 19.225)
+		(end 103.4 19.3)
+		(width 0.2)
+		(layer "B.Cu")
+		(net "GND")
 	)
 	(segment
@@
 		(size 0.6)
 		(drill 0.3)
+		(layers "F.Cu" "B.Cu")
+		(net "GND")
+	)
+	(via
+		(at 102 15.225)
+		(size 0.6)
+		(drill 0.3)
+		(layers "F.Cu" "B.Cu")
+		(net "GND")
+	)
+	(via
+		(at 103.4 19.3)
+		(size 0.6)
+		(drill 0.3)
