File: hardware/coupon/rev-a/staging/paired-charger-local-routing-trial-114mm.kicad_pcb (KiCad board)
At the start: 6 copper layers, 114 x 32.5 mm, 483 parts, among them J1 USB4505-03-0-A, J2 S2B-PH-SM4-TB, SW1 EVQP7J01P, SW2 JS202011JCQN, U1 TLC59581RTQT, U11 SN74LVC1G04DBVR, U17 SN74LVC1G11DBVR, U2 74HC4514PW,118, U23 SN74LVC1G06DBVR, U24 SN74LVC2G17DBVR, U25 SN74LVC2G17DBVR, U29 TPS70933DBVR, U3 ESP32-S3-WROOM-1U-N16R8, U31 TUSB320LAIRWBR, U32 TS3USB31ERSER, U33 TPD4E05U06DQAR, U34 TPS3808G01DBVR, U35 MAX17048G+T10, U36 TPS631000DRLR, U37 TPS63020DSJT, U38 2.5V shunt, U39 TMP390A2DRLR, U40 SN74AUP1G125DBVR, U41 BQ24074RGTR, U42 SN74AUP1G125DBVR, U43 SN74AUP1G125DBVR, U44 TPS259474ARPWR, U45 TPS259474ARPWR, U46 TCA9517ADGKR, U47 TPS3823A-33DBVR, U48 SN74LVC1G04DSFR, U49 SN74LVC1G74RSER, U50 SN74LVC1G74RSER, U51 SN74LVC1G11DRYR, U52 SN74LVC1G08DSFR, U53 TLV6700DSER, U54 SN74LVC2G00DCUR, U55 SN74LVC2G08DCUR

Commit message: Route staged USB rails across 114 mm charger study
Routing:
- net CHARGER_IN_DRAFT: track 2.29 -> 21.2 mm, vias 0 -> 3
- net VBUS_CONNECTOR: track 0.00 -> 16.4 mm, vias 0 -> 3
- net +5V_USB: track 0.00 -> 10.2 mm, vias 0 -> 2
Changed lines of the file:
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@@
+	)
+	(segment
+		(start 100.5 15)
+		(end 100.5 17)
+		(width 0.2)
+		(layer "B.Cu")
+		(net "+5V_USB")
+	)
+	(segment
+		(start 100.5 17)
+		(end 105.35 17)
+		(width 0.2)
+		(layer "In4.Cu")
+		(net "+5V_USB")
+	)
+	(segment
+		(start 100.5 19)
+		(end 100.5 20.5)
+		(width 0.2)
+		(layer "B.Cu")
+		(net "CHARGER_IN_DRAFT")
+	)
+	(segment
+		(start 100.5 20.5)
+		(end 100.7 20.8)
+		(width 0.2)
+		(layer "B.Cu")
+		(net "CHARGER_IN_DRAFT")
+	)
+	(segment
+		(start 100.7 20.8)
+		(end 103.7 20.8)
+		(width 0.2)
+		(layer "In4.Cu")
+		(net "CHARGER_IN_DRAFT")
+	)
+	(segment
+		(start 101 12.5)
+		(end 104.5 12.5)
+		(width 0.2)
+		(layer "In4.Cu")
+		(net "VBUS_CONNECTOR")
+	)
+	(segment
+		(start 101 15)
+		(end 101 12.5)
+		(width 0.2)
+		(layer "B.Cu")
+		(net "VBUS_CONNECTOR")
+	)
+	(segment
+		(start 101 17.5)
+		(end 100.5 17)
+		(width 0.2)
+		(layer "B.Cu")
+		(net "+5V_USB")
+	)
+	(segment
+		(start 101 19)
+		(end 101 17.5)
+		(width 0.2)
+		(layer "B.Cu")
+		(net "+5V_USB")
+	)
+	(segment
+		(start 103.7 20.8)
+		(end 105.5 19)
+		(width 0.2)
+		(layer "In4.Cu")
+		(net "CHARGER_IN_DRAFT")
+	)
+	(segment
+		(start 104.5 12.5)
+		(end 105.2 13.2)
+		(width 0.2)
+		(layer "In4.Cu")
+		(net "VBUS_CONNECTOR")
 	)
 	(segment
@@
 	)
 	(segment
+		(start 105.2 13.2)
+		(end 105.2 14)
+		(width 0.2)
+		(layer "B.Cu")
+		(net "VBUS_CONNECTOR")
+	)
+	(segment
+		(start 105.2 13.2)
+		(end 105.85 13.85)
+		(width 0.2)
+		(layer "F.Cu")
+		(net "VBUS_CONNECTOR")
+	)
+	(segment
 		(start 105.3 26)
 		(end 110 25.5)
@@
 	)
 	(segment
+		(start 105.35 17)
+		(end 105.55 16.8)
+		(width 0.2)
+		(layer "In4.Cu")
+		(net "+5V_USB")
+	)
+	(segment
 		(start 105.4 27.6)
 		(end 106 27)
@@
 	)
 	(segment
+		(start 105.5 19)
+		(end 104.65 19)
+		(width 0.2)
+		(layer "B.Cu")
+		(net "CHARGER_IN_DRAFT")
+	)
+	(segment
+		(start 105.5 19)
+		(end 105.5 23.5)
+		(width 0.2)
+		(layer "In4.Cu")
+		(net "CHARGER_IN_DRAFT")
+	)
+	(segment
+		(start 105.5 23.5)
+		(end 109.5 27.5)
+		(width 0.2)
+		(layer "In4.Cu")
+		(net "CHARGER_IN_DRAFT")
+	)
+	(segment
 		(start 105.5 24.75)
 		(end 106.25 25.5)
@@
 	)
 	(segment
+		(start 105.55 16.8)
+		(end 105.3 16)
+		(width 0.2)
+		(layer "B.Cu")
+		(net "+5V_USB")
+	)
+	(segment
+		(start 105.85 13.85)
+		(end 107.25 13.85)
+		(width 0.2)
+		(layer "F.Cu")
+		(net "VBUS_CONNECTOR")
+	)
+	(segment
 		(start 106 27)
 		(end 107.5 26.65)
@@
 	)
 	(segment
+		(start 107.2 15.2)
+		(end 105.2 13.2)
+		(width 0.2)
+		(layer "In4.Cu")
+		(net "VBUS_CONNECTOR")
+	)
+	(segment
+		(start 107.2 18.65)
+		(end 107.2 15.2)
+		(width 0.2)
+		(layer "In4.Cu")
+		(net "VBUS_CONNECTOR")
+	)
+	(segment
+		(start 107.25 18.65)
+		(end 107.2 18.65)
+		(width 0.2)
+		(layer "F.Cu")
+		(net "VBUS_CONNECTOR")
+	)
+	(segment
 		(start 108.55 28.75)
 		(end 109 28.3)
@@
 	)
 	(segment
+		(start 109.5 27.5)
+		(end 109 27.5)
+		(width 0.2)
+		(layer "B.Cu")
+		(net "CHARGER_IN_DRAFT")
+	)
+	(segment
 		(start 110 25.5)
 		(end 110.5 25)
@@
 	)
 	(via
+		(at 100.5 17)
+		(size 0.6)
+		(drill 0.3)
+		(layers "F.Cu" "B.Cu")
+		(net "+5V_USB")
+	)
+	(via
+		(at 100.7 20.8)
+		(size 0.6)
+		(drill 0.3)
+		(layers "F.Cu" "B.Cu")
+		(net "CHARGER_IN_DRAFT")
+	)
+	(via
+		(at 101 12.5)
+		(size 0.6)
+		(drill 0.3)
+		(layers "F.Cu" "B.Cu")
+		(net "VBUS_CONNECTOR")
+	)
+	(via
+		(at 105.2 13.2)
+		(size 0.6)
+		(drill 0.3)
+		(layers "F.Cu" "B.Cu")
+		(net "VBUS_CONNECTOR")
+	)
+	(via
 		(at 105.3 26)
 		(size 0.6)
@@
 	)
 	(via
+		(at 105.5 19)
+		(size 0.6)
+		(drill 0.3)
+		(layers "F.Cu" "B.Cu")
+		(net "CHARGER_IN_DRAFT")
+	)
+	(via
+		(at 105.55 16.8)
+		(size 0.6)
+		(drill 0.3)
+		(layers "F.Cu" "B.Cu")
+		(net "+5V_USB")
+	)
+	(via
+		(at 107.2 18.65)
+		(size 0.6)
+		(drill 0.3)
+		(layers "F.Cu" "B.Cu")
+		(net "VBUS_CONNECTOR")
+	)
+	(via
+		(at 109.5 27.5)
+		(size 0.6)
+		(drill 0.3)
+		(layers "F.Cu" "B.Cu")
+		(net "CHARGER_IN_DRAFT")
+	)
+	(via

Commit message: Center battery sensors in 114 mm placement study
Parts:
- moved PAIR15 86.8 mm to (25.5, 25.0)
- moved TP10 86.0 mm to (97.0, 9.25)
- moved PAIR14 83.3 mm to (112.2, 24.5)
- moved TP5 82.8 mm to (104.0, 30.0)
- moved PAIR09 82.3 mm to (104.2, 21.5)
- moved U36 81.2 mm to (18.6, 7.25)
- moved U54 76.6 mm to (93.1, 19.4)
- moved TP2 76.5 mm to (21.3, 20.0)
- moved TP33 74.9 mm to (96.0, 30.0)
- moved C73 74.5 mm to (89.8, 21.5)
- moved U32 74.0 mm to (26.0, 28.2)
- moved U53 72.4 mm to (11.8, 4.38)
- moved C42 70.8 mm to (97.1, 27.8)
- moved U35 70.8 mm to (93.0, 28.1)
- moved C43 70.8 mm to (22.4, 28.0)
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Routing:
- net GND: track 0.00 -> 49.5 mm, vias 0 -> 8

Commit message: Extend 114 mm charger trial ground returns
Routing:
- net GND: track 49.5 -> 72.9 mm, vias 8 -> 15
Changed lines of the file:
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@@
+	)
+	(segment
+		(start 103.7 15.45)
+		(end 103.8 13.5)
+		(width 0.2)
+		(layer "In3.Cu")
+		(net "GND")
+	)
+	(segment
+		(start 103.7 16)
+		(end 103.7 15.45)
+		(width 0.2)
+		(layer "B.Cu")
+		(net "GND")
 	)
 	(segment
@@
 	)
 	(segment
+		(start 108 23.1)
+		(end 106.8 23.1)
+		(width 0.2)
+		(layer "In2.Cu")
+		(net "GND")
+	)
+	(segment
+		(start 108 23.85)
+		(end 108 23.1)
+		(width 0.2)
+		(layer "B.Cu")
+		(net "GND")
+	)
+	(segment
 		(start 108.55 28.75)
 		(end 109 28.3)
@@
 	)
 	(segment
+		(start 109 23.1)
+		(end 106.8 23.1)
+		(width 0.2)
+		(layer "In2.Cu")
+		(net "GND")
+	)
+	(segment
+		(start 109 23.85)
+		(end 109 23.1)
+		(width 0.2)
+		(layer "B.Cu")
+		(net "GND")
+	)
+	(segment
 		(start 109 28.3)
 		(end 109 26.65)
@@
 		(net "CHARGER_ILIM")
 	)
+	(segment
+		(start 96.85 15.3)
+		(end 99.1 15.2)
+		(width 0.2)
+		(layer "In3.Cu")
+		(net "GND")
+	)
+	(segment
+		(start 96.85 16)
+		(end 96.85 15.3)
+		(width 0.2)
+		(layer "B.Cu")
+		(net "GND")
+	)
+	(segment
+		(start 96.85 19)
+		(end 96.85 19.6)
+		(width 0.2)
+		(layer "B.Cu")
+		(net "GND")
+	)
+	(segment
+		(start 96.85 19.6)
+		(end 99 19.225)
+		(width 0.2)
+		(layer "In3.Cu")
+		(net "GND")
+	)
+	(segment
+		(start 99 19.225)
+		(end 103.1 19)
+		(width 0.2)
+		(layer "In3.Cu")
+		(net "GND")
+	)
+	(segment
+		(start 99.1 15.2)
+		(end 103.7 15.45)
+		(width 0.2)
+		(layer "In3.Cu")
+		(net "GND")
+	)
+	(segment
+		(start 99.85 15.225)
+		(end 99.1 15.2)
+		(width 0.2)
+		(layer "B.Cu")
+		(net "GND")
+	)
+	(segment
+		(start 99.85 19.225)
+		(end 99 19.225)
+		(width 0.2)
+		(layer "B.Cu")
+		(net "GND")
+	)
 	(via
 		(at 100.5 17)
@@
 	)
 	(via
+		(at 103.7 15.45)
+		(size 0.6)
+		(drill 0.3)
+		(layers "F.Cu" "B.Cu")
+		(net "GND")
+	)
+	(via
 		(at 103.8 13.5)
 		(size 0.6)
@@
 	)
 	(via
+		(at 108 23.1)
+		(size 0.6)
+		(drill 0.3)
+		(layers "F.Cu" "B.Cu")
+		(net "GND")
+	)
+	(via
+		(at 109 23.1)
+		(size 0.6)
+		(drill 0.3)
+		(layers "F.Cu" "B.Cu")
+		(net "GND")
+	)
+	(via
 		(at 109.5 27.5)
 		(size 0.6)
@@
 		(size 0.6)
 		(drill 0.3)
+		(layers "F.Cu" "B.Cu")
+		(net "GND")
+	)
+	(via
+		(at 96.85 15.3)
+		(size 0.6)
+		(drill 0.3)
+		(layers "F.Cu" "B.Cu")
+		(net "GND")
+	)
+	(via
+		(at 96.85 19.6)
+		(size 0.6)
+		(drill 0.3)
+		(layers "F.Cu" "B.Cu")
+		(net "GND")
+	)
+	(via
+		(at 99 19.225)
+		(size 0.6)
+		(drill 0.3)
+		(layers "F.Cu" "B.Cu")
+		(net "GND")
+	)
+	(via
+		(at 99.1 15.2)
+		(size 0.6)
+		(drill 0.3)

Commit message: Route both eFuse timing capacitors on 114 mm study
Routing:
- net E1_DVDT: track 0.00 -> 3.50 mm
- net E0_DVDT: track 0.00 -> 2.38 mm
Changed lines of the file:
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@@
+	)
+	(segment
+		(start 100.025 20)
+		(end 100.025 19.875)
+		(width 0.2)
+		(layer "B.Cu")
+		(net "E1_DVDT")
 	)
 	(segment
@@
 	)
 	(segment
+		(start 97.65 16)
+		(end 100.025 15.875)
+		(width 0.2)
+		(layer "B.Cu")
+		(net "E0_DVDT")
+	)
+	(segment
+		(start 97.65 19)
+		(end 97.65 20)
+		(width 0.2)
+		(layer "B.Cu")
+		(net "E1_DVDT")
+	)
+	(segment
+		(start 97.65 20)
+		(end 100.025 20)
+		(width 0.2)
+		(layer "B.Cu")
+		(net "E1_DVDT")
+	)
+	(segment

Commit message: Route E0 control network on 114 mm trial
Routing:
- net E0_OVLO: track 0.00 -> 13.9 mm, vias 0 -> 3
- net E0_EN: track 0.00 -> 10.6 mm, vias 0 -> 2
- net VBUS_CONNECTOR: track 16.4 -> 26.1 mm, vias 3 -> 4
- net GND: track 72.9 -> 82.0 mm
- net E0_ILM: track 0.00 -> 2.87 mm
Changed lines of the file:
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@@
+	)
+	(segment
+		(start 100 11.5)
+		(end 102.5 11.5)
+		(width 0.2)
+		(layer "In2.Cu")
+		(net "E0_EN")
 	)
 	(segment
@@
 	)
 	(segment
+		(start 101.65 14.775)
+		(end 102.5 14.775)
+		(width 0.2)
+		(layer "B.Cu")
+		(net "E0_OVLO")
+	)
+	(segment
 		(start 101.65 18.775)
 		(end 102.2 18.775)
@@
 	)
 	(segment
+		(start 102.5 11.5)
+		(end 102.5 13.4)
+		(width 0.2)
+		(layer "In2.Cu")
+		(net "E0_EN")
+	)
+	(segment
+		(start 102.5 13.4)
+		(end 101.65 14.3)
+		(width 0.2)
+		(layer "B.Cu")
+		(net "E0_EN")
+	)
+	(segment
 		(start 102.95 24.75)
 		(end 102.95 26.75)
@@
 	)
 	(segment
+		(start 95.9 12)
+		(end 100 11.5)
+		(width 0.2)
+		(layer "In2.Cu")
+		(net "E0_EN")
+	)
+	(segment
+		(start 95.9 17.5)
+		(end 102.5 14.775)
+		(width 0.2)
+		(layer "In2.Cu")
+		(net "E0_OVLO")
+	)
+	(segment
+		(start 96 15.225)
+		(end 103.7 15.45)
+		(width 0.2)
+		(layer "In3.Cu")
+		(net "GND")
+	)
+	(segment
+		(start 96.75 12)
+		(end 95.9 12)
+		(width 0.2)
+		(layer "B.Cu")
+		(net "E0_EN")
+	)
+	(segment
+		(start 96.75 14)
+		(end 96 15.225)
+		(width 0.2)
+		(layer "B.Cu")
+		(net "GND")
+	)
+	(segment
+		(start 96.75 17.5)
+		(end 95.9 17.5)
+		(width 0.2)
+		(layer "B.Cu")
+		(net "E0_OVLO")
+	)
+	(segment
+		(start 96.75 20.75)
+		(end 96.85 19.6)
+		(width 0.2)
+		(layer "B.Cu")
+		(net "GND")
+	)
+	(segment
+		(start 96.75 22.5)
+		(end 96.75 20.75)
+		(width 0.2)
+		(layer "B.Cu")
+		(net "GND")
+	)
+	(segment
 		(start 96.85 15.3)
-		(end 99.1 15.2)
+		(end 96 15.225)
 		(width 0.2)
 		(layer "In3.Cu")
@@
 	)
 	(segment
+		(start 97.75 12)
+		(end 101 12.5)
+		(width 0.2)
+		(layer "B.Cu")
+		(net "VBUS_CONNECTOR")
+	)
+	(segment
+		(start 97.75 14)
+		(end 97.75 14.775)
+		(width 0.2)
+		(layer "B.Cu")
+		(net "E0_ILM")
+	)
+	(segment
+		(start 97.75 14.775)
+		(end 99.85 14.775)
+		(width 0.2)
+		(layer "B.Cu")
+		(net "E0_ILM")
+	)
+	(segment
+		(start 97.75 17.5)
+		(end 98.5 17.5)
+		(width 0.2)
+		(layer "B.Cu")
+		(net "VBUS_CONNECTOR")
+	)
+	(segment
+		(start 97.75 20.75)
+		(end 98.6 20.75)
+		(width 0.2)
+		(layer "B.Cu")
+		(net "E0_OVLO")
+	)
+	(segment
+		(start 98.5 17.5)
+		(end 101 12.5)
+		(width 0.2)
+		(layer "In4.Cu")
+		(net "VBUS_CONNECTOR")
+	)
+	(segment
+		(start 98.6 20.75)
+		(end 95.9 17.5)
+		(width 0.2)
+		(layer "In2.Cu")
+		(net "E0_OVLO")
+	)
+	(segment
 		(start 99 19.225)
 		(end 103.1 19)
@@
 	)
 	(segment
-		(start 99.1 15.2)
-		(end 103.7 15.45)
-		(width 0.2)
-		(layer "In3.Cu")
-		(net "GND")
-	)
-	(segment
 		(start 99.85 15.225)
-		(end 99.1 15.2)
+		(end 96 15.225)
 		(width 0.2)
 		(layer "B.Cu")
@@
 	)
 	(via
+		(at 102.5 13.4)
+		(size 0.6)
+		(drill 0.3)
+		(layers "F.Cu" "B.Cu")
+		(net "E0_EN")
+	)
+	(via
+		(at 102.5 14.775)
+		(size 0.6)
+		(drill 0.3)
+		(layers "F.Cu" "B.Cu")
+		(net "E0_OVLO")
+	)
+	(via
 		(at 103 28.5)
 		(size 0.6)
@@
 	)
 	(via
+		(at 95.9 12)
+		(size 0.6)
+		(drill 0.3)
+		(layers "F.Cu" "B.Cu")
+		(net "E0_EN")
+	)
+	(via
+		(at 95.9 17.5)
+		(size 0.6)
+		(drill 0.3)
+		(layers "F.Cu" "B.Cu")
+		(net "E0_OVLO")
+	)
+	(via
+		(at 96 15.225)
+		(size 0.6)
+		(drill 0.3)
+		(layers "F.Cu" "B.Cu")
+		(net "GND")
+	)
+	(via
 		(at 96.85 15.3)
 		(size 0.6)
@@
 	)
 	(via
+		(at 98.5 17.5)
+		(size 0.6)
+		(drill 0.3)
+		(layers "F.Cu" "B.Cu")
+		(net "VBUS_CONNECTOR")
+	)
+	(via
+		(at 98.6 20.75)
+		(size 0.6)
+		(drill 0.3)
+		(layers "F.Cu" "B.Cu")
+		(net "E0_OVLO")
+	)
+	(via
 		(at 99 19.225)
 		(size 0.6)
 		(drill 0.3)
-		(layers "F.Cu" "B.Cu")
-		(net "GND")
-	)
-	(via
-		(at 99.1 15.2)
-		(size 0.6)
-		(drill 0.3)

Commit message: Stage battery and switch power paths on 114 mm trial
Routing:
- net +BAT_PROTECTED_DRAFT: track 2.61 -> 108.0 mm, vias 0 -> 3
- net +SYS_APP_IN_DRAFT: track 7.34 -> 110.9 mm, vias 2 -> 3
- net GND: track 82.0 -> 170.2 mm, vias 15 -> 16
Changed lines of the file:
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@@
+	)
+	(segment
+		(start 106.85 25)
+		(end 106.85 25.5)
+		(width 0.2)
+		(layer "B.Cu")
+		(net "+BAT_PROTECTED_DRAFT")
 	)
 	(segment
@@
 	)
 	(segment
+		(start 108.25 25.25)
+		(end 108 23.85)
+		(width 0.2)
+		(layer "B.Cu")
+		(net "GND")
+	)
+	(segment
 		(start 108.55 28.75)
 		(end 109 28.3)
@@
 	)
 	(segment
+		(start 109.65 25.5)
+		(end 109.65 25)
+		(width 0.2)
+		(layer "B.Cu")
+		(net "+SYS_APP_IN_DRAFT")
+	)
+	(segment
 		(start 110 25.5)
 		(end 110.5 25)
@@
 	)
 	(segment
+		(start 22.5 1.8)
+		(end 30 1.8)
+		(width 0.5)
+		(layer "In2.Cu")
+		(net "GND")
+	)
+	(segment
+		(start 23.85 2.5)
+		(end 22.5 1.8)
+		(width 0.2)
+		(layer "B.Cu")
+		(net "GND")
+	)
+	(segment
+		(start 25.85 2.5)
+		(end 27 3)
+		(width 0.2)
+		(layer "B.Cu")
+		(net "+BAT_PROTECTED_DRAFT")
+	)
+	(segment
+		(start 27 3)
+		(end 105.5 24.75)
+		(width 0.5)
+		(layer "In1.Cu")
+		(net "+BAT_PROTECTED_DRAFT")
+	)
+	(segment
+		(start 30 1.8)
+		(end 103 28.5)
+		(width 0.5)
+		(layer "In2.Cu")
+		(net "GND")
+	)
+	(segment
+		(start 5.3 1.4)
+		(end 6.5 1.4)
+		(width 0.2)
+		(layer "B.Cu")
+		(net "+SYS_APP_IN_DRAFT")
+	)
+	(segment
+		(start 5.3 3.8)
+		(end 6.5 4.8)
+		(width 0.2)
+		(layer "B.Cu")
+		(net "+BAT_PROTECTED_DRAFT")
+	)
+	(segment
+		(start 6.5 1.4)
+		(end 105.3 26)
+		(width 0.5)
+		(layer "In3.Cu")
+		(net "+SYS_APP_IN_DRAFT")
+	)
+	(segment
+		(start 6.5 4.8)
+		(end 27 3)
+		(width 0.5)
+		(layer "In1.Cu")
+		(net "+BAT_PROTECTED_DRAFT")
+	)
+	(segment
 		(start 95.9 12)
 		(end 100 11.5)
@@
 	)
 	(via
+		(at 105.5 24.75)
+		(size 0.6)
+		(drill 0.3)
+		(layers "F.Cu" "B.Cu")
+		(net "+BAT_PROTECTED_DRAFT")
+	)
+	(via
 		(at 105.55 16.8)
 		(size 0.6)
@@
 	)
 	(via
+		(at 22.5 1.8)
+		(size 0.6)
+		(drill 0.3)
+		(layers "F.Cu" "B.Cu")
+		(net "GND")
+	)
+	(via
+		(at 27 3)
+		(size 0.6)
+		(drill 0.3)
+		(layers "F.Cu" "B.Cu")
+		(net "+BAT_PROTECTED_DRAFT")
+	)
+	(via
+		(at 6.5 1.4)
+		(size 0.6)
+		(drill 0.3)
+		(layers "F.Cu" "B.Cu")
+		(net "+SYS_APP_IN_DRAFT")
+	)
+	(via
+		(at 6.5 4.8)
+		(size 0.6)
+		(drill 0.3)
+		(layers "F.Cu" "B.Cu")
+		(net "+BAT_PROTECTED_DRAFT")
+	)
+	(via

Commit message: Connect USB shell returns in 114 mm routing trial
Routing:
- net GND: track 170.2 -> 182.1 mm
Changed lines of the file:
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@@
+	)
+	(segment
+		(start 108.4 10.63)
+		(end 107.5 12.3)
+		(width 0.2)
+		(layer "In3.Cu")
+		(net "GND")
+	)
+	(segment
+		(start 108.4 10.63)
+		(end 112.4 10.63)
+		(width 0.2)
+		(layer "In3.Cu")
+		(net "GND")
+	)
+	(segment
+		(start 108.4 21.87)
+		(end 106.8 23.1)
+		(width 0.2)
+		(layer "In2.Cu")
+		(net "GND")
+	)
+	(segment
+		(start 108.4 21.87)
+		(end 112.4 21.87)
+		(width 0.2)
+		(layer "In2.Cu")
+		(net "GND")
 	)
 	(segment

Commit message: Route E1 current-limit network on 114 mm trial
Routing:
- net E1_ILM: track 0.00 -> 13.5 mm, vias 0 -> 2
Changed lines of the file:
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@@
+	)
+	(segment
+		(start 97.7 19.5)
+		(end 98.5 18.4)
+		(width 0.2)
+		(layer "In4.Cu")
+		(net "E1_ILM")
+	)
+	(segment
+		(start 97.7 21.6)
+		(end 97.7 19.5)
+		(width 0.2)
+		(layer "In4.Cu")
+		(net "E1_ILM")
 	)
 	(segment
@@
 	)
 	(segment
+		(start 97.75 22.5)
+		(end 98.5 22.5)
+		(width 0.2)
+		(layer "B.Cu")
+		(net "E1_ILM")
+	)
+	(segment
 		(start 98.5 17.5)
 		(end 101 12.5)
@@
 	)
 	(segment
+		(start 98.5 18.4)
+		(end 99.2 18.4)
+		(width 0.2)
+		(layer "B.Cu")
+		(net "E1_ILM")
+	)
+	(segment
+		(start 98.5 22.5)
+		(end 98.5 25.5)
+		(width 0.2)
+		(layer "B.Cu")
+		(net "E1_ILM")
+	)
+	(segment
+		(start 98.5 25.5)
+		(end 99 24.5)
+		(width 0.2)
+		(layer "In4.Cu")
+		(net "E1_ILM")
+	)
+	(segment
 		(start 98.6 20.75)
 		(end 95.9 17.5)
@@
 	)
 	(segment
+		(start 99 22.5)
+		(end 97.7 21.6)
+		(width 0.2)
+		(layer "In4.Cu")
+		(net "E1_ILM")
+	)
+	(segment
+		(start 99 24.5)
+		(end 99 22.5)
+		(width 0.2)
+		(layer "In4.Cu")
+		(net "E1_ILM")
+	)
+	(segment
+		(start 99.2 18.4)
+		(end 99.4 18.775)
+		(width 0.2)
+		(layer "B.Cu")
+		(net "E1_ILM")
+	)
+	(segment
+		(start 99.4 18.775)
+		(end 99.85 18.775)
+		(width 0.2)
+		(layer "B.Cu")
+		(net "E1_ILM")
+	)
+	(segment
 		(start 99.85 15.225)
 		(end 96 15.225)
@@
 	)
 	(via
+		(at 98.5 18.4)
+		(size 0.6)
+		(drill 0.3)
+		(layers "F.Cu" "B.Cu")
+		(net "E1_ILM")
+	)
+	(via
+		(at 98.5 25.5)
+		(size 0.6)
+		(drill 0.3)
+		(layers "F.Cu" "B.Cu")
+		(net "E1_ILM")
+	)
+	(via
