File: hardware/coupon/rev-a/staging/paired-charger-local-routing-trial-114mm.kicad_pcb (KiCad board)
At the start: 6 copper layers, 114 x 32.5 mm, 483 parts, among them J1 USB4505-03-0-A, J2 S2B-PH-SM4-TB, SW1 EVQP7J01P, SW2 JS202011JCQN, U1 TLC59581RTQT, U11 SN74LVC1G04DBVR, U17 SN74LVC1G11DBVR, U2 74HC4514PW,118, U23 SN74LVC1G06DBVR, U24 SN74LVC2G17DBVR, U25 SN74LVC2G17DBVR, U29 TPS70933DBVR, U3 ESP32-S3-WROOM-1U-N16R8, U31 TUSB320LAIRWBR, U32 TS3USB31ERSER, U33 TPD4E05U06DQAR, U34 TPS3808G01DBVR, U35 MAX17048G+T10, U36 TPS631000DRLR, U37 TPS63020DSJT, U38 2.5V shunt, U39 TMP390A2DRLR, U40 SN74AUP1G125DBVR, U41 BQ24074RGTR, U42 SN74AUP1G125DBVR, U43 SN74AUP1G125DBVR, U44 TPS259474ARPWR, U45 TPS259474ARPWR, U46 TCA9517ADGKR, U47 TPS3823A-33DBVR, U48 SN74LVC1G04DSFR, U49 SN74LVC1G74RSER, U50 SN74LVC1G74RSER, U51 SN74LVC1G11DRYR, U52 SN74LVC1G08DSFR, U53 TLV6700DSER, U54 SN74LVC2G00DCUR, U55 SN74LVC2G08DCUR

Commit message: Place and route local USB logic LDO bypass capacitors
Parts:
- moved C32 55.3 mm to (89.2, 10.5)
- moved TP14 55.3 mm to (34.0, 1.00)
- moved C30 47.9 mm to (97.2, 9.00)
- moved TP10 22.1 mm to (93.0, 31.0)
Routing:
- net GND: track 253.2 -> 267.9 mm, vias 22 -> 24
- net +5V_USB: track 20.3 -> 27.0 mm
- net +3V3_USB: track 132.7 -> 134.0 mm
Changed lines of the file:
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@@
 	(footprint "rgb-badge-coupon:C_Murata_GRM18_0603"
 		(layer "B.Cu")
-		(at 34.75 1 180)
+		(at 89.25 10.5 180)
 		(descr "GRM18 0603 reflow land pattern, midpoint of Murata recommended ranges; SPDX-License-Identifier: CERN-OHL-S-2.0")
 		(property "Reference" "C32"
@@
 	(footprint "rgb-badge-coupon:TestPoint_Pad_D1.0mm"
 		(layer "B.Cu")
-		(at 88.501262 10.500001 180)
+		(at 34.001262 1.000001 180)
 		(descr "Bare 1.0 mm copper probe pad; no purchased component or solder paste. SPDX-License-Identifier: CERN-OHL-S-2.0")
 		(property "Reference" "TP14"
@@
 	(footprint "rgb-badge-coupon:C_Murata_GRM15_0402"
 		(layer "B.Cu")
-		(at 49.75 2.75 180)
+		(at 97.25 9 180)
 		(descr "Manufacturer range-based reflow land pattern; SPDX-License-Identifier: CERN-OHL-S-2.0")
 		(property "Reference" "C30"
@@
 	(footprint "rgb-badge-coupon:TestPoint_Pad_D1.0mm"
 		(layer "B.Cu")
-		(at 97.001262 9.250001 180)
+		(at 93.001262 31.000001 180)
 		(descr "Bare 1.0 mm copper probe pad; no purchased component or solder paste. SPDX-License-Identifier: CERN-OHL-S-2.0")
 		(property "Reference" "TP10"
@@
 	)
 	(segment
+		(start 88.45 10.5)
+		(end 88.45 11.4)
+		(width 0.2)
+		(layer "B.Cu")
+		(net "GND")
+	)
+	(segment
+		(start 88.45 11.4)
+		(end 95.8 10.875)
+		(width 0.2)
+		(layer "In3.Cu")
+		(net "GND")
+	)
+	(segment
 		(start 90 14.175)
 		(end 91.2 14.175)
@@
 	)
 	(segment
+		(start 90.05 10.5)
+		(end 91.2 9.925)
+		(width 0.2)
+		(layer "B.Cu")
+		(net "+3V3_USB")
+	)
+	(segment
 		(start 91.2 16.075)
 		(end 93 14.3)
@@
 	)
 	(segment
+		(start 94 10.875)
+		(end 95.8 10.875)
+		(width 0.2)
+		(layer "In3.Cu")
+		(net "GND")
+	)
+	(segment
 		(start 94 14.7)
 		(end 96 15.22)
@@
 	)
 	(segment
+		(start 94 8.3)
+		(end 94 9.925)
+		(width 0.2)
+		(layer "B.Cu")
+		(net "+5V_USB")
+	)
+	(segment
+		(start 94 9.15)
+		(end 94 10.875)
+		(width 0.2)
+		(layer "In3.Cu")
+		(net "GND")
+	)
+	(segment
+		(start 94 9.925)
+		(end 94.8 9.925)
+		(width 0.2)
+		(layer "B.Cu")
+		(net "+5V_USB")
+	)
+	(segment
 		(start 94.8 10.875)
 		(end 95.8 10.875)
@@
 	)
 	(segment
+		(start 96.2 9.15)
+		(end 94 9.15)
+		(width 0.2)
+		(layer "In3.Cu")
+		(net "GND")
+	)
+	(segment
 		(start 96.75 12)
 		(end 95.9 12)
@@
 	)
 	(segment
+		(start 96.85 9)
+		(end 96.2 9.15)
+		(width 0.2)
+		(layer "B.Cu")
+		(net "GND")
+	)
+	(segment
 		(start 97 9.925)
 		(end 100.5 17)
@@
 	)
 	(segment
+		(start 97.65 8.3)
+		(end 94 8.3)
+		(width 0.2)
+		(layer "B.Cu")
+		(net "+5V_USB")
+	)
+	(segment
+		(start 97.65 9)
+		(end 97.65 8.3)
+		(width 0.2)
+		(layer "B.Cu")
+		(net "+5V_USB")
+	)
+	(segment
 		(start 97.7 19.5)
 		(end 98.5 18.4)
@@
 	)
 	(via
+		(at 88.45 11.4)
+		(size 0.6)
+		(drill 0.3)
+		(layers "F.Cu" "B.Cu")
+		(net "GND")
+	)
+	(via
 		(at 91.2 14.175)
 		(size 0.6)
@@
 		(size 0.6)
 		(drill 0.3)
+		(layers "F.Cu" "B.Cu")
+		(net "GND")
+	)
+	(via
+		(at 96.2 9.15)
+		(size 0.6)
+		(drill 0.3)

Commit message: Route local USB qualification links on 114 mm study
Routing:
- net +3V3_USB: track 134.0 -> 155.2 mm, vias 8 -> 10
- net USB_CC_HIGH: track 0.00 -> 13.4 mm, vias 0 -> 2
- net USB_VBUS_VALID: track 0.00 -> 11.1 mm, vias 0 -> 2
- net GND: track 267.9 -> 278.5 mm, vias 24 -> 25
- net USB_LOGIC_READY: track 0.00 -> 8.65 mm

Commit message: Route supervisor reset bias and shared pull-down returns
Routing:
- net USB_RAW_LOGIC_READY: track 5.96 -> 93.5 mm, vias 2 -> 4
- net GND: track 278.5 -> 356.3 mm, vias 25 -> 26
- net +3V3_USB: track 155.2 -> 162.8 mm
Changed lines of the file:
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@@
+	)
+	(segment
+		(start 20.45 14.6)
+		(end 20.45 11.675)
+		(width 0.2)
+		(layer "B.Cu")
+		(net "+3V3_USB")
 	)
 	(segment
@@
 	)
 	(segment
+		(start 24.05 12.625)
+		(end 29.05 12.625)
+		(width 0.2)
+		(layer "B.Cu")
+		(net "GND")
+	)
+	(segment
+		(start 24.05 13.575)
+		(end 24.05 14.6)
+		(width 0.2)
+		(layer "B.Cu")
+		(net "+3V3_USB")
+	)
+	(segment
+		(start 24.05 14.6)
+		(end 20.45 14.6)
+		(width 0.2)
+		(layer "B.Cu")
+		(net "+3V3_USB")
+	)
+	(segment
 		(start 24.05 15.925)
 		(end 25.05 15.925)
@@
 		(start 24.55 15.425)
 		(end 25.05 15.925)
+		(width 0.2)
+		(layer "In2.Cu")
+		(net "USB_RAW_LOGIC_READY")
+	)
+	(segment
+		(start 24.55 7)
+		(end 24.55 11.675)
+		(width 0.2)
+		(layer "In4.Cu")
+		(net "USB_RAW_LOGIC_READY")
+	)
+	(segment
+		(start 24.55 9)
+		(end 24.55 11.675)
 		(width 0.2)
 		(layer "In2.Cu")
@@
 	)
 	(segment
+		(start 29.5 10.25)
+		(end 29.5 9)
+		(width 0.2)
+		(layer "B.Cu")
+		(net "USB_RAW_LOGIC_READY")
+	)
+	(segment
+		(start 29.5 9)
+		(end 24.55 9)
+		(width 0.2)
+		(layer "In2.Cu")
+		(net "USB_RAW_LOGIC_READY")
+	)
+	(segment
 		(start 29.9 11.675)
 		(end 30 9.5)
@@
 	)
 	(segment
+		(start 31.75 10.25)
+		(end 29.5 10.25)
+		(width 0.2)
+		(layer "B.Cu")
+		(net "USB_RAW_LOGIC_READY")
+	)
+	(segment
 		(start 32.75 10.25)
 		(end 32.75 9.5)
@@
 	)
 	(segment
+		(start 58.5 6.5)
+		(end 76.5 6.5)
+		(width 0.2)
+		(layer "B.Cu")
+		(net "GND")
+	)
+	(segment
+		(start 58.5 8.75)
+		(end 58.5 6.5)
+		(width 0.2)
+		(layer "B.Cu")
+		(net "GND")
+	)
+	(segment
 		(start 59.2 16)
 		(end 76.3 16)
+		(width 0.2)
+		(layer "B.Cu")
+		(net "GND")
+	)
+	(segment
+		(start 59.25 7.25)
+		(end 59.25 6.5)
+		(width 0.2)
+		(layer "B.Cu")
+		(net "GND")
+	)
+	(segment
+		(start 59.25 8.75)
+		(end 58.5 8.75)
 		(width 0.2)
 		(layer "B.Cu")
@@
 	)
 	(segment
+		(start 60.25 8)
+		(end 76.5 8)
+		(width 0.2)
+		(layer "B.Cu")
+		(net "USB_RAW_LOGIC_READY")
+	)
+	(segment
+		(start 60.25 8.75)
+		(end 60.25 8)
+		(width 0.2)
+		(layer "B.Cu")
+		(net "USB_RAW_LOGIC_READY")
+	)
+	(segment
+		(start 61.75 7.25)
+		(end 61.75 6.5)
+		(width 0.2)
+		(layer "B.Cu")
+		(net "GND")
+	)
+	(segment
+		(start 64.25 7.25)
+		(end 64.25 6.5)
+		(width 0.2)
+		(layer "B.Cu")
+		(net "GND")
+	)
+	(segment
+		(start 66.75 7.25)
+		(end 66.75 6.5)
+		(width 0.2)
+		(layer "B.Cu")
+		(net "GND")
+	)
+	(segment
 		(start 67.5 13.5)
 		(end 69.25 11.75)
@@
 	)
 	(segment
+		(start 69.25 7.25)
+		(end 69.25 6.5)
+		(width 0.2)
+		(layer "B.Cu")
+		(net "GND")
+	)
+	(segment
 		(start 70.25 10.25)
 		(end 70.25 11.4)
@@
 	)
 	(segment
+		(start 71.75 7.25)
+		(end 71.75 6.5)
+		(width 0.2)
+		(layer "B.Cu")
+		(net "GND")
+	)
+	(segment
 		(start 71.75 9.5)
 		(end 75.25 9.5)
@@
 	)
 	(segment
+		(start 74.25 7.25)
+		(end 74.25 6.5)
+		(width 0.2)
+		(layer "B.Cu")
+		(net "GND")
+	)
+	(segment
 		(start 75 14.4)
 		(end 76.25 10.25)
@@
 	)
 	(segment
+		(start 76.5 6.5)
+		(end 77 6.25)
+		(width 0.2)
+		(layer "B.Cu")
+		(net "GND")
+	)
+	(segment
+		(start 76.5 8)
+		(end 77.5 7.75)
+		(width 0.2)
+		(layer "B.Cu")
+		(net "USB_RAW_LOGIC_READY")
+	)
+	(segment
+		(start 77 6.25)
+		(end 31 6.25)
+		(width 0.2)
+		(layer "In2.Cu")
+		(net "GND")
+	)
+	(segment
 		(start 77.5 12.1)
 		(end 77.5 12.5)
@@
 	)
 	(segment
+		(start 77.5 7)
+		(end 24.55 7)
+		(width 0.2)
+		(layer "In4.Cu")
+		(net "USB_RAW_LOGIC_READY")
+	)
+	(segment
+		(start 77.5 7.75)
+		(end 77.5 7)
+		(width 0.2)
+		(layer "In4.Cu")
+		(net "USB_RAW_LOGIC_READY")
+	)
+	(segment
 		(start 77.5 9.5)
 		(end 77.5 12.5)
@@
 	)
 	(via
+		(at 29.5 9)
+		(size 0.6)
+		(drill 0.3)
+		(layers "F.Cu" "B.Cu")
+		(net "USB_RAW_LOGIC_READY")
+	)
+	(via
 		(at 29.9 11.675)
 		(size 0.6)
@@
 	)
 	(via
+		(at 77 6.25)
+		(size 0.6)
+		(drill 0.3)
+		(layers "F.Cu" "B.Cu")
+		(net "GND")
+	)
+	(via
 		(at 77.5 12.5)
 		(size 0.6)
@@
 	)
 	(via
+		(at 77.5 7.75)
+		(size 0.6)
+		(drill 0.3)
+		(layers "F.Cu" "B.Cu")
+		(net "USB_RAW_LOGIC_READY")
+	)
+	(via
