File: hardware/coupon/rev-a/staging/paired-charger-placement-only-114mm.kicad_pcb (KiCad board)
At the start: 6 copper layers, 114 x 32.5 mm, 483 parts, among them J1 USB4505-03-0-A, J2 S2B-PH-SM4-TB, SW1 EVQP7J01P, SW2 JS202011JCQN, U1 TLC59581RTQT, U11 SN74LVC1G04DBVR, U17 SN74LVC1G11DBVR, U2 74HC4514PW,118, U23 SN74LVC1G06DBVR, U24 SN74LVC2G17DBVR, U25 SN74LVC2G17DBVR, U29 TPS70933DBVR, U3 ESP32-S3-WROOM-1U-N16R8, U31 TUSB320LAIRWBR, U32 TS3USB31ERSER, U33 TPD4E05U06DQAR, U34 TPS3808G01DBVR, U35 MAX17048G+T10, U36 TPS631000DRLR, U37 TPS63020DSJT, U38 2.5V shunt, U39 TMP390A2DRLR, U40 SN74AUP1G125DBVR, U41 BQ24074RGTR, U42 SN74AUP1G125DBVR, U43 SN74AUP1G125DBVR, U44 TPS259474ARPWR, U45 TPS259474ARPWR, U46 TCA9517ADGKR, U47 TPS3823A-33DBVR, U48 SN74LVC1G04DSFR, U49 SN74LVC1G74RSER, U50 SN74LVC1G74RSER, U51 SN74LVC1G11DRYR, U52 SN74LVC1G08DSFR, U53 TLV6700DSER, U54 SN74LVC2G00DCUR, U55 SN74LVC2G08DCUR

Commit message: Center battery sensors in 114 mm placement study
Parts:
- moved PAIR15 86.8 mm to (25.5, 25.0)
- moved TP10 86.0 mm to (97.0, 9.25)
- moved PAIR14 83.3 mm to (112.2, 24.5)
- moved TP5 82.8 mm to (104.0, 30.0)
- moved PAIR09 82.3 mm to (104.2, 21.5)
- moved U36 81.2 mm to (18.6, 7.25)
- moved U54 76.6 mm to (93.1, 19.4)
- moved TP2 76.5 mm to (21.3, 20.0)
- moved TP33 74.9 mm to (96.0, 30.0)
- moved C73 74.5 mm to (89.8, 21.5)
- moved U32 74.0 mm to (26.0, 28.2)
- moved U53 72.4 mm to (11.8, 4.38)
- moved C42 70.8 mm to (97.1, 27.8)
- moved U35 70.8 mm to (93.0, 28.1)
- moved C43 70.8 mm to (22.4, 28.0)
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
Commit message: Place and route local USB logic LDO bypass capacitors
Parts:
- moved C32 55.3 mm to (89.2, 10.5)
- moved TP14 55.3 mm to (34.0, 1.00)
- moved C30 47.9 mm to (97.2, 9.00)
- moved TP10 22.1 mm to (93.0, 31.0)
Changed lines of the file:
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@@
 	(footprint "rgb-badge-coupon:C_Murata_GRM15_0402"
 		(layer "B.Cu")
-		(at 49.75 2.75 180)
+		(at 97.25 9 180)
 		(descr "Manufacturer range-based reflow land pattern; SPDX-License-Identifier: CERN-OHL-S-2.0")
 		(property "Reference" "C30"
@@
 	(footprint "rgb-badge-coupon:C_Murata_GRM18_0603"
 		(layer "B.Cu")
-		(at 34.75 1 180)
+		(at 89.25 10.5 180)
 		(descr "GRM18 0603 reflow land pattern, midpoint of Murata recommended ranges; SPDX-License-Identifier: CERN-OHL-S-2.0")
 		(property "Reference" "C32"
@@
 	(footprint "rgb-badge-coupon:TestPoint_Pad_D1.0mm"
 		(layer "B.Cu")
-		(at 97.001262 9.250001 180)
+		(at 93.001262 31.000001 180)
 		(descr "Bare 1.0 mm copper probe pad; no purchased component or solder paste. SPDX-License-Identifier: CERN-OHL-S-2.0")
 		(property "Reference" "TP10"
@@
 	(footprint "rgb-badge-coupon:TestPoint_Pad_D1.0mm"
 		(layer "B.Cu")
-		(at 88.501262 10.500001 180)
+		(at 34.001262 1.000001 180)
 		(descr "Bare 1.0 mm copper probe pad; no purchased component or solder paste. SPDX-License-Identifier: CERN-OHL-S-2.0")
 		(property "Reference" "TP14"
