File: hardware/coupon/rev-a/staging/onsemi-row-placement-trial-114mm.kicad_pcb (KiCad board)
At the start: 6 copper layers, 114 x 32.5 mm, 483 parts, among them J1 USB4505-03-0-A, J2 S2B-PH-SM4-TB, SW1 EVQP7J01P, SW2 JS202011JCQN, U1 TLC59581RTQT, U11 SN74LVC1G04DBVR, U17 SN74LVC1G11DBVR, U2 74HC4514PW,118, U23 SN74LVC1G06DBVR, U24 SN74LVC2G17DBVR, U25 SN74LVC2G17DBVR, U29 TPS70933DBVR, U3 ESP32-S3-WROOM-1U-N16R8, U31 TUSB320LAIRWBR, U32 TS3USB31ERSER, U33 TPD4E05U06DQAR, U34 TPS3808G01DBVR, U35 MAX17048G+T10, U36 TPS631000DRLR, U37 TPS63020DSJT, U38 2.5V shunt, U39 TMP390A2DRLR, U40 SN74AUP1G125DBVR, U41 BQ24074RGTR, U42 SN74AUP1G125DBVR, U43 SN74AUP1G125DBVR, U44 TPS259474ARPWR, U45 TPS259474ARPWR, U46 TCA9517ADGKR, U47 TPS3823A-33DBVR, U48 SN74LVC1G04DSFR, U49 SN74LVC1G74RSER, U50 SN74LVC1G74RSER, U51 SN74LVC1G11DRYR, U52 SN74LVC1G08DSFR, U53 TLV6700DSER, U54 SN74LVC2G00DCUR, U55 SN74LVC2G08DCUR

Commit message: Route USB logic LDO output and return on study board
Routing:
- net GND: track 250.4 -> 253.2 mm, vias 21 -> 22
- net +3V3_USB: track 130.5 -> 132.7 mm, vias 7 -> 8

Commit message: Route protected USB rail to logic LDO input
Routing:
- net +5V_USB: track 10.2 -> 20.3 mm, vias 2 -> 3

Commit message: Place and route local USB logic LDO bypass capacitors
Parts:
- moved C32 55.3 mm to (89.2, 10.5)
- moved TP14 55.3 mm to (34.0, 1.00)
- moved C30 47.9 mm to (97.2, 9.00)
- moved TP10 22.1 mm to (93.0, 31.0)
Routing:
- net GND: track 253.2 -> 267.9 mm, vias 22 -> 24
- net +5V_USB: track 20.3 -> 27.0 mm
- net +3V3_USB: track 132.7 -> 134.0 mm

Commit message: Route local USB qualification links on 114 mm study
Routing:
- net +3V3_USB: track 134.0 -> 155.2 mm, vias 8 -> 10
- net USB_CC_HIGH: track 0.00 -> 13.4 mm, vias 0 -> 2
- net USB_VBUS_VALID: track 0.00 -> 11.1 mm, vias 0 -> 2
- net GND: track 267.9 -> 278.5 mm, vias 24 -> 25
- net USB_LOGIC_READY: track 0.00 -> 8.65 mm

Commit message: Route supervisor reset bias and shared pull-down returns
Routing:
- net USB_RAW_LOGIC_READY: track 5.96 -> 93.5 mm, vias 2 -> 4
- net GND: track 278.5 -> 356.3 mm, vias 25 -> 26
- net +3V3_USB: track 155.2 -> 162.8 mm
