File: hardware/coupon/rev-a/staging/led-qt-uniform-2p2-row-bank-onsemi-trial-114mm.kicad_pcb (KiCad board)
At the start: 6 copper layers, 114 x 32.5 mm, 483 parts, among them J1 USB4505-03-0-A, J2 S2B-PH-SM4-TB, SW1 EVQP7J01P, SW2 JS202011JCQN, U1 TLC59581RTQT, U11 SN74LVC1G04DBVR, U17 SN74LVC1G11DBVR, U2 74HC4514PW,118, U23 SN74LVC1G06DBVR, U24 SN74LVC2G17DBVR, U25 SN74LVC2G17DBVR, U29 TPS70933DBVR, U3 ESP32-S3-WROOM-1U-N16R8, U31 TUSB320LAIRWBR, U32 TS3USB31ERSER, U33 TPD4E05U06DQAR, U34 TPS3808G01DBVR, U35 MAX17048G+T10, U36 TPS631000DRLR, U37 TPS63020DSJT, U38 2.5V shunt, U39 TMP390A2DRLR, U40 SN74AUP1G125DBVR, U41 BQ24074RGTR, U42 SN74AUP1G125DBVR, U43 SN74AUP1G125DBVR, U44 TPS259474ARPWR, U45 TPS259474ARPWR, U46 TCA9517ADGKR, U47 TPS3823A-33DBVR, U48 SN74LVC1G04DSFR, U49 SN74LVC1G74RSER, U50 SN74LVC1G74RSER, U51 SN74LVC1G11DRYR, U52 SN74LVC1G08DSFR, U53 TLV6700DSER, U54 SN74LVC2G00DCUR, U55 SN74LVC2G08DCUR

Commit message: Connect first matrix colour trunk to TLC59581
Routing:
- net COL_08_R: track 29.2 -> 54.1 mm, vias 16 -> 20
Changed lines of the file:
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@@
 	)
 	(segment
+		(start 58.675 0.65)
+		(end 82.6 4.75)
+		(width 0.2)
+		(layer "In4.Cu")
+		(net "COL_08_R")
+	)
+	(segment
+		(start 58.675 1.225)
+		(end 58.675 0.65)
+		(width 0.2)
+		(layer "In1.Cu")
+		(net "COL_08_R")
+	)
+	(segment
 		(start 58.675 1.225)
 		(end 58.675 3.175)
@@
 	)
 	(via micro
+		(at 58.675 0.65)
+		(size 0.3)
+		(drill 0.1)
+		(layers "In1.Cu" "In2.Cu")
+		(net "COL_08_R")
+	)
+	(via micro
+		(at 58.675 0.65)
+		(size 0.3)
+		(drill 0.1)
+		(layers "In2.Cu" "In3.Cu")
+		(net "COL_08_R")
+	)
+	(via micro
+		(at 58.675 0.65)
+		(size 0.3)
+		(drill 0.1)
+		(layers "In3.Cu" "In4.Cu")
+		(net "COL_08_R")
+	)
+	(via micro
 		(at 58.675 1.225)
 		(size 0.3)
@@
 		(net "ROW_03_A")
 	)
+	(via micro
+		(at 82.6 4.75)
+		(size 0.3)
+		(drill 0.1)
+		(layers "In4.Cu" "B.Cu")
+		(net "COL_08_R")
+	)
 	(embedded_fonts no)

Commit message: Stagger four colour-driver fanouts on row-bank study
Routing:
- net COL_13_R: track 29.2 -> 48.4 mm, vias 16 -> 20
- net COL_14_R: track 29.2 -> 47.8 mm, vias 16 -> 20
- net COL_15_B: track 29.2 -> 47.4 mm, vias 16 -> 20
Changed lines of the file:
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@@
 	)
 	(segment
+		(start 69.675 0.65)
+		(end 88.25 1.1)
+		(width 0.2)
+		(layer "In4.Cu")
+		(net "COL_13_R")
+	)
+	(segment
+		(start 69.675 1.225)
+		(end 69.675 0.65)
+		(width 0.2)
+		(layer "In1.Cu")
+		(net "COL_13_R")
+	)
+	(segment
 		(start 69.675 1.225)
 		(end 69.675 3.175)
@@
 	(segment
 		(start 71.875 1.225)
+		(end 71.875 1.25)
+		(width 0.2)
+		(layer "In1.Cu")
+		(net "COL_14_R")
+	)
+	(segment
+		(start 71.875 1.225)
 		(end 71.875 3.175)
 		(width 0.2)
@@
 	)
 	(segment
+		(start 71.875 1.25)
+		(end 90.4 2.25)
+		(width 0.2)
+		(layer "In4.Cu")
+		(net "COL_14_R")
+	)
+	(segment
 		(start 71.875 10.975)
 		(end 71.875 12.925)
@@
 	)
 	(segment
+		(start 72.675 1.85)
+		(end 90.4 4.75)
+		(width 0.2)
+		(layer "In4.Cu")
+		(net "COL_15_B")
+	)
+	(segment
 		(start 72.675 10.975)
 		(end 73.375 11.375)
@@
 	(segment
 		(start 72.675 2.025)
+		(end 72.675 1.85)
+		(width 0.2)
+		(layer "In1.Cu")
+		(net "COL_15_B")
+	)
+	(segment
+		(start 72.675 2.025)
 		(end 72.675 3.975)
 		(width 0.2)
@@
 	)
 	(via micro
+		(at 69.675 0.65)
+		(size 0.3)
+		(drill 0.1)
+		(layers "In1.Cu" "In2.Cu")
+		(net "COL_13_R")
+	)
+	(via micro
+		(at 69.675 0.65)
+		(size 0.3)
+		(drill 0.1)
+		(layers "In2.Cu" "In3.Cu")
+		(net "COL_13_R")
+	)
+	(via micro
+		(at 69.675 0.65)
+		(size 0.3)
+		(drill 0.1)
+		(layers "In3.Cu" "In4.Cu")
+		(net "COL_13_R")
+	)
+	(via micro
 		(at 69.675 1.225)
 		(size 0.3)
@@
 	)
 	(via micro
+		(at 71.875 1.25)
+		(size 0.3)
+		(drill 0.1)
+		(layers "In1.Cu" "In2.Cu")
+		(net "COL_14_R")
+	)
+	(via micro
+		(at 71.875 1.25)
+		(size 0.3)
+		(drill 0.1)
+		(layers "In2.Cu" "In3.Cu")
+		(net "COL_14_R")
+	)
+	(via micro
+		(at 71.875 1.25)
+		(size 0.3)
+		(drill 0.1)
+		(layers "In3.Cu" "In4.Cu")
+		(net "COL_14_R")
+	)
+	(via micro
 		(at 71.875 10.975)
 		(size 0.3)
@@
 	)
 	(via micro
+		(at 72.675 1.85)
+		(size 0.3)
+		(drill 0.1)
+		(layers "In1.Cu" "In2.Cu")
+		(net "COL_15_B")
+	)
+	(via micro
+		(at 72.675 1.85)
+		(size 0.3)
+		(drill 0.1)
+		(layers "In2.Cu" "In3.Cu")
+		(net "COL_15_B")
+	)
+	(via micro
+		(at 72.675 1.85)
+		(size 0.3)
+		(drill 0.1)
+		(layers "In3.Cu" "In4.Cu")
+		(net "COL_15_B")
+	)
+	(via micro
 		(at 72.675 11.775)
 		(size 0.3)
@@
 		(net "COL_08_R")
 	)
+	(via micro
+		(at 88.25 1.1)
+		(size 0.3)
+		(drill 0.1)
+		(layers "In4.Cu" "B.Cu")
+		(net "COL_13_R")
+	)
+	(via micro
+		(at 90.4 2.25)
+		(size 0.3)
+		(drill 0.1)
+		(layers "In4.Cu" "B.Cu")
+		(net "COL_14_R")
+	)
+	(via micro
+		(at 90.4 4.75)
+		(size 0.3)
+		(drill 0.1)
+		(layers "In4.Cu" "B.Cu")
+		(net "COL_15_B")
+	)
 	(embedded_fonts no)

Commit message: Add lower-edge 1010 colour fanout examples
Routing:
- net COL_00_R: track 29.2 -> 97.0 mm, vias 16 -> 20
- net COL_07_R: track 29.2 -> 81.6 mm, vias 16 -> 20
Changed lines of the file:
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@@
 	)
 	(segment
+		(start 42.8 31.3)
+		(end 42.8 31.85)
+		(width 0.2)
+		(layer "In1.Cu")
+		(net "COL_00_R")
+	)
+	(segment
+		(start 42.8 31.85)
+		(end 82.1 31.85)
+		(width 0.2)
+		(layer "In4.Cu")
+		(net "COL_00_R")
+	)
+	(segment
 		(start 42.8 4)
 		(end 42.8 5.95)
@@
 	)
 	(segment
+		(start 56.45 31.3)
+		(end 56.45 31.85)
+		(width 0.2)
+		(layer "In1.Cu")
+		(net "COL_07_R")
+	)
+	(segment
+		(start 56.45 31.85)
+		(end 73.75 31.85)
+		(width 0.2)
+		(layer "In2.Cu")
+		(net "COL_07_R")
+	)
+	(segment
 		(start 56.45 4)
 		(end 56.45 5.95)
@@
 	)
 	(segment
+		(start 73.75 31.85)
+		(end 74.25 31.25)
+		(width 0.2)
+		(layer "In2.Cu")
+		(net "COL_07_R")
+	)
+	(segment
 		(start 74.075 1.225)
 		(end 74.075 3.175)
@@
 	)
 	(segment
+		(start 74.25 31.25)
+		(end 75.15 31.25)
+		(width 0.2)
+		(layer "In2.Cu")
+		(net "COL_07_R")
+	)
+	(segment
 		(start 74.7 10.4)
 		(end 77.25 11.9)
@@
 	)
 	(segment
+		(start 75.15 31.25)
+		(end 75.65 31.85)
+		(width 0.2)
+		(layer "In2.Cu")
+		(net "COL_07_R")
+	)
+	(segment
+		(start 75.65 31.85)
+		(end 82.1 31.85)
+		(width 0.2)
+		(layer "In2.Cu")
+		(net "COL_07_R")
+	)
+	(segment
 		(start 76.675 11.9)
 		(end 77.25 11.9)
@@
 		(net "ROW_01_A")
 	)
+	(segment
+		(start 82.1 31.85)
+		(end 82.6 6.25)
+		(width 0.2)
+		(layer "In2.Cu")
+		(net "COL_07_R")
+	)
+	(segment
+		(start 82.1 31.85)
+		(end 90.4 5.25)
+		(width 0.2)
+		(layer "In4.Cu")
+		(net "COL_00_R")
+	)
 	(via
 		(at 77.25 11.9)
@@
 	)
 	(via micro
+		(at 42.8 31.85)
+		(size 0.3)
+		(drill 0.1)
+		(layers "In1.Cu" "In2.Cu")
+		(net "COL_00_R")
+	)
+	(via micro
+		(at 42.8 31.85)
+		(size 0.3)
+		(drill 0.1)
+		(layers "In2.Cu" "In3.Cu")
+		(net "COL_00_R")
+	)
+	(via micro
+		(at 42.8 31.85)
+		(size 0.3)
+		(drill 0.1)
+		(layers "In3.Cu" "In4.Cu")
+		(net "COL_00_R")
+	)
+	(via micro
 		(at 42.8 4)
 		(size 0.3)
@@
 	)
 	(via micro
+		(at 56.45 31.85)
+		(size 0.3)
+		(drill 0.1)
+		(layers "In1.Cu" "In2.Cu")
+		(net "COL_07_R")
+	)
+	(via micro
 		(at 56.45 4)
 		(size 0.3)
@@
 	)
 	(via micro
+		(at 82.6 6.25)
+		(size 0.3)
+		(drill 0.1)
+		(layers "In2.Cu" "In3.Cu")
+		(net "COL_07_R")
+	)
+	(via micro
+		(at 82.6 6.25)
+		(size 0.3)
+		(drill 0.1)
+		(layers "In3.Cu" "In4.Cu")
+		(net "COL_07_R")
+	)
+	(via micro
+		(at 82.6 6.25)
+		(size 0.3)
+		(drill 0.1)
+		(layers "In4.Cu" "B.Cu")
+		(net "COL_07_R")
+	)
+	(via micro
 		(at 88.25 1.1)
 		(size 0.3)
@@
 		(net "COL_15_B")
 	)
+	(via micro
+		(at 90.4 5.25)
+		(size 0.3)
+		(drill 0.1)
+		(layers "In4.Cu" "B.Cu")
+		(net "COL_00_R")
+	)
 	(embedded_fonts no)
