File: hardware/coupon/rev-a/staging/led-native-control-trial-114mm.kicad_pcb (KiCad board)
At the start: 6 copper layers, 114 x 32.5 mm, 483 parts, among them J1 USB4505-03-0-A, J2 S2B-PH-SM4-TB, SW1 EVQP7J01P, SW2 JS202011JCQN, U1 TLC59581RTQT, U11 SN74LVC1G04DBVR, U17 SN74LVC1G11DBVR, U2 74HC4514PW,118, U23 SN74LVC1G06DBVR, U24 SN74LVC2G17DBVR, U25 SN74LVC2G17DBVR, U29 TPS70933DBVR, U3 ESP32-S3-WROOM-1U-N16R8, U31 TUSB320LAIRWBR, U32 TS3USB31ERSER, U33 TPD4E05U06DQAR, U34 TPS3808G01DBVR, U35 MAX17048G+T10, U36 TPS631000DRLR, U37 TPS63020DSJT, U38 2.5V shunt, U39 TMP390A2DRLR, U40 SN74AUP1G125DBVR, U41 BQ24074RGTR, U42 SN74AUP1G125DBVR, U43 SN74AUP1G125DBVR, U44 TPS259474ARPWR, U45 TPS259474ARPWR, U46 TCA9517ADGKR, U47 TPS3823A-33DBVR, U48 SN74LVC1G04DSFR, U49 SN74LVC1G74RSER, U50 SN74LVC1G74RSER, U51 SN74LVC1G11DRYR, U52 SN74LVC1G08DSFR, U53 TLV6700DSER, U54 SN74LVC2G00DCUR, U55 SN74LVC2G08DCUR

Commit message: Complete gauge clock and route arm and USB charge-request controls
Routing:
- net GAUGE_I2C_SCL: track 37.8 -> 124.3 mm, vias 2 -> 11
- net ROW_ARM: track 0.00 -> 74.9 mm, vias 0 -> 4
- net USB_CHARGE_REQ: track 87.6 -> 129.3 mm, vias 9 -> 12

Commit message: Reserve R28 ground escape and add exact native grid screening
Routing:
- net ROW_SEL_04: track 101.9 -> 103.9 mm
- net GND: track 115.8 -> 115.9 mm, vias 490 -> 493
Changed lines of the file:
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@@
 	(segment
 		(start 38.6 7.25)
-		(end 54 7.25)
+		(end 40.5 7.25)
 		(width 0.2)
 		(layer "In4.Cu")
@@
 	)
 	(segment
+		(start 40.5 6.25)
+		(end 42.3 6.25)
+		(width 0.2)
+		(layer "In4.Cu")
+		(net "ROW_SEL_04")
+	)
+	(segment
+		(start 40.5 7.25)
+		(end 40.5 6.25)
+		(width 0.2)
+		(layer "In4.Cu")
+		(net "ROW_SEL_04")
+	)
+	(segment
 		(start 40.6 0.649999)
 		(end 42.8 0.649999)
@@
 	)
 	(segment
+		(start 41.75 7.25)
+		(end 41.85 7.2)
+		(width 0.2)
+		(layer "B.Cu")
+		(net "GND")
+	)
+	(segment
 		(start 41.85 2.75)
 		(end 41.85 2.75)
@@
 	)
 	(segment
+		(start 42.3 6.25)
+		(end 42.3 7.25)
+		(width 0.2)
+		(layer "In4.Cu")
+		(net "ROW_SEL_04")
+	)
+	(segment
+		(start 42.3 7.25)
+		(end 54 7.25)
+		(width 0.2)
+		(layer "In4.Cu")
+		(net "ROW_SEL_04")
+	)
+	(segment
 		(start 42.35 11.75)
 		(end 42.35 12.1)
@@
 		(size 0.3)
 		(drill 0.1)
+		(layers "In4.Cu" "B.Cu")
+		(net "GND")
+	)
+	(via micro
+		(at 41.85 7.2)
+		(size 0.3)
+		(drill 0.1)
+		(layers "In2.Cu" "In3.Cu")
+		(net "GND")
+	)
+	(via micro
+		(at 41.85 7.2)
+		(size 0.3)
+		(drill 0.1)
+		(layers "In3.Cu" "In4.Cu")
+		(net "GND")
+	)
+	(via micro
+		(at 41.85 7.2)
+		(size 0.3)
+		(drill 0.1)
