File: hardware/coupon/rev-a/staging/led-routing-progress-trial-114mm.kicad_pcb (KiCad board)
At the start: 6 copper layers, 114 x 32.5 mm, 483 parts, among them J1 USB4505-03-0-A, J2 S2B-PH-SM4-TB, SW1 EVQP7J01P, SW2 JS202011JCQN, U1 TLC59581RTQT, U11 SN74LVC1G04DBVR, U17 SN74LVC1G11DBVR, U2 74HC4514PW,118, U23 SN74LVC1G06DBVR, U24 SN74LVC2G17DBVR, U25 SN74LVC2G17DBVR, U29 TPS70933DBVR, U3 ESP32-S3-WROOM-1U-N16R8, U31 TUSB320LAIRWBR, U32 TS3USB31ERSER, U33 TPD4E05U06DQAR, U34 TPS3808G01DBVR, U35 MAX17048G+T10, U36 TPS631000DRLR, U37 TPS63020DSJT, U38 2.5V shunt, U39 TMP390A2DRLR, U40 SN74AUP1G125DBVR, U41 BQ24074RGTR, U42 SN74AUP1G125DBVR, U43 SN74AUP1G125DBVR, U44 TPS259474ARPWR, U45 TPS259474ARPWR, U46 TCA9517ADGKR, U47 TPS3823A-33DBVR, U48 SN74LVC1G04DSFR, U49 SN74LVC1G74RSER, U50 SN74LVC1G74RSER, U51 SN74LVC1G11DRYR, U52 SN74LVC1G08DSFR, U53 TLV6700DSER, U54 SN74LVC2G00DCUR, U55 SN74LVC2G08DCUR

Commit message: Complete row addresses and C67 ground at 82 opens
Routing:
- net ROW_A1: track 8.97 -> 137.9 mm, vias 0 -> 44
- net GND: track 158.8 -> 177.9 mm, vias 621 -> 625
