File: hardware/coupon/rev-a/staging/vled-converter.kicad_sch (KiCad schematic)
At the start: 13 parts, among them U37 TPS63020DSJT

Commit message: Correct all six exact Murata capacitor lands and preserve 59-edge routing
Parts:
- C44, C45: footprint rgb-badge-coupon:C_Murata_GRM18_0603 -> rgb-badge-coupon:C_Murata_GRM188R60J106ME47_0603
Changed lines of the file:
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@@
 (property "Reference" "C44" (at 76.200 49.530 0) (effects (font (size 1.27 1.27))))
 (property "Value" "10u 6.3V X5R" (at 76.200 52.070 0) (effects (font (size 1.27 1.27))))
-(property "Footprint" "rgb-badge-coupon:C_Murata_GRM18_0603" (at 76.200 55.880 0) (effects (font (size 1.27 1.27)) (hide yes)))
+(property "Footprint" "rgb-badge-coupon:C_Murata_GRM188R60J106ME47_0603" (at 76.200 55.880 0) (effects (font (size 1.27 1.27)) (hide yes)))
 (property "Datasheet" "https://pim.murata.com/en-global/pim/details/?partNum=GRM188R60J106ME47D" (at 76.200 55.880 0) (effects (font (size 1.27 1.27)) (hide yes)))
 (property "Manufacturer" "Murata" (at 76.200 55.880 0) (effects (font (size 1.27 1.27)) (hide yes)))
@@
 (property "Reference" "C45" (at 76.200 67.310 0) (effects (font (size 1.27 1.27))))
 (property "Value" "10u 6.3V X5R" (at 76.200 69.850 0) (effects (font (size 1.27 1.27))))
-(property "Footprint" "rgb-badge-coupon:C_Murata_GRM18_0603" (at 76.200 73.660 0) (effects (font (size 1.27 1.27)) (hide yes)))
+(property "Footprint" "rgb-badge-coupon:C_Murata_GRM188R60J106ME47_0603" (at 76.200 73.660 0) (effects (font (size 1.27 1.27)) (hide yes)))
 (property "Datasheet" "https://pim.murata.com/en-global/pim/details/?partNum=GRM188R60J106ME47D" (at 76.200 73.660 0) (effects (font (size 1.27 1.27)) (hide yes)))
 (property "Manufacturer" "Murata" (at 76.200 73.660 0) (effects (font (size 1.27 1.27)) (hide yes)))
